File: hardware/KiCad/LivSynth_0v1/LFO.kicad_sch (KiCad schematic)
At the start: 19 parts, among them Q5 2N3904, Q6 2N3904, Q7 2N3904, U2 TL074, U3 TL074

Commit message: 0v1 Ready for Production
Parts:
- renumbered C33 to C23, D6 to D2, D9 to D6, Q6 to Q1, Q5 to Q15, Q7 to Q16, R30 to R19, R31 to R22, R27 to R4, R32 to R40, R29 to R41, R24 to R5, R28 to R61, R26 to R64, R25 to R68, RV4 to RV9, U2 to U3, U3 to U8
Changed lines of the file:
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@@
   (symbol (lib_id "Amplifier_Operational:TL074") (at 154.94 78.74 0) (unit 4)
     (in_bom yes) (on_board yes)
-    (property "Reference" "U2" (id 0) (at 154.94 69.85 0))
+    (property "Reference" "U3" (id 0) (at 154.94 69.85 0))
     (property "Value" "TL074" (id 1) (at 154.94 72.39 0))
     (property "Footprint" "Package_SO:SOIC-14_3.9x8.7mm_P1.27mm" (id 2) (at 153.67 76.2 0)
@@
   (symbol (lib_id "Device:R") (at 139.7 76.2 90) (unit 1)
     (in_bom yes) (on_board yes) (fields_autoplaced)
-    (property "Reference" "R28" (id 0) (at 139.7 69.85 90))
+    (property "Reference" "R61" (id 0) (at 139.7 69.85 90))
     (property "Value" "80K" (id 1) (at 139.7 72.39 90))
     (property "Footprint" "Resistor_THT:R_Axial_DIN0207_L6.3mm_D2.5mm_P7.62mm_Horizontal" (id 2) (at 139.7 77.978 90)
@@
   (symbol (lib_id "Device:R") (at 165.1 129.54 0) (unit 1)
     (in_bom yes) (on_board yes) (fields_autoplaced)
-    (property "Reference" "R32" (id 0) (at 167.64 128.2699 0)
+    (property "Reference" "R40" (id 0) (at 167.64 128.2699 0)
       (effects (font (size 1.27 1.27)) (justify left))
     )
@@
   (symbol (lib_id "Device:C") (at 124.46 62.23 90) (unit 1)
     (in_bom yes) (on_board yes) (fields_autoplaced)
-    (property "Reference" "C33" (id 0) (at 124.46 54.61 90))
+    (property "Reference" "C23" (id 0) (at 124.46 54.61 90))
     (property "Value" "100n" (id 1) (at 124.46 57.15 90))
     (property "Footprint" "Capacitor_THT:C_Rect_L7.2mm_W2.5mm_P5.00mm_FKS2_FKP2_MKS2_MKP2" (id 2) (at 128.27 61.2648 0)
@@
   (symbol (lib_id "Device:R") (at 217.17 49.53 0) (unit 1)
     (in_bom yes) (on_board yes) (fields_autoplaced)
-    (property "Reference" "R24" (id 0) (at 219.075 48.2599 0)
+    (property "Reference" "R5" (id 0) (at 219.075 48.2599 0)
       (effects (font (size 1.27 1.27)) (justify left))
     )
@@
   (symbol (lib_id "Device:R") (at 201.93 62.23 270) (unit 1)
     (in_bom yes) (on_board yes) (fields_autoplaced)
-    (property "Reference" "R27" (id 0) (at 201.93 56.515 90))
+    (property "Reference" "R4" (id 0) (at 201.93 56.515 90))
     (property "Value" "100K" (id 1) (at 201.93 59.055 90))
     (property "Footprint" "Resistor_THT:R_Axial_DIN0207_L6.3mm_D2.5mm_P7.62mm_Horizontal" (id 2) (at 201.93 60.452 90)
@@
   (symbol (lib_id "Device:R_Potentiometer") (at 107.315 73.66 0) (unit 1)
     (in_bom yes) (on_board yes) (fields_autoplaced)
-    (property "Reference" "RV4" (id 0) (at 104.775 72.3899 0)
+    (property "Reference" "RV9" (id 0) (at 104.775 72.3899 0)
       (effects (font (size 1.27 1.27)) (justify right))
     )
@@
   (symbol (lib_id "Transistor_BJT:2N3904") (at 97.155 85.09 90) (unit 1)
     (in_bom yes) (on_board yes)
-    (property "Reference" "Q7" (id 0) (at 101.6 85.725 90))
+    (property "Reference" "Q16" (id 0) (at 101.6 85.725 90))
     (property "Value" "2N3904" (id 1) (at 102.87 88.265 90))
     (property "Footprint" "Package_TO_SOT_THT:TO-92_Inline" (id 2) (at 99.06 80.01 0)
@@
   (symbol (lib_id "Device:R") (at 133.985 117.475 270) (unit 1)
     (in_bom yes) (on_board yes) (fields_autoplaced)
-    (property "Reference" "R31" (id 0) (at 133.985 111.76 90))
+    (property "Reference" "R22" (id 0) (at 133.985 111.76 90))
     (property "Value" "100R" (id 1) (at 133.985 114.3 90))
     (property "Footprint" "Resistor_THT:R_Axial_DIN0207_L6.3mm_D2.5mm_P7.62mm_Horizontal" (id 2) (at 133.985 115.697 90)
@@
   (symbol (lib_id "Device:R") (at 140.335 49.53 90) (unit 1)
     (in_bom yes) (on_board yes) (fields_autoplaced)
-    (property "Reference" "R25" (id 0) (at 140.335 43.18 90))
+    (property "Reference" "R68" (id 0) (at 140.335 43.18 90))
     (property "Value" "1M" (id 1) (at 140.335 45.72 90))
     (property "Footprint" "Resistor_THT:R_Axial_DIN0207_L6.3mm_D2.5mm_P7.62mm_Horizontal" (id 2) (at 140.335 51.308 90)
@@
   (symbol (lib_id "Amplifier_Operational:TL074") (at 125.095 76.2 0) (mirror x) (unit 3)
     (in_bom yes) (on_board yes)
-    (property "Reference" "U2" (id 0) (at 125.095 67.31 0))
+    (property "Reference" "U3" (id 0) (at 125.095 67.31 0))
     (property "Value" "TL074" (id 1) (at 125.095 69.85 0))
     (property "Footprint" "Package_SO:SOIC-14_3.9x8.7mm_P1.27mm" (id 2) (at 123.825 78.74 0)
@@
   (symbol (lib_id "Transistor_BJT:2N3904") (at 214.63 62.23 0) (unit 1)
     (in_bom yes) (on_board yes)
-    (property "Reference" "Q6" (id 0) (at 219.71 60.9599 0)
+    (property "Reference" "Q1" (id 0) (at 219.71 60.9599 0)
       (effects (font (size 1.27 1.27)) (justify left))
     )
@@
   (symbol (lib_id "Transistor_BJT:2N3904") (at 97.155 62.23 270) (unit 1)
     (in_bom yes) (on_board yes)
-    (property "Reference" "Q5" (id 0) (at 101.6 62.23 90))
+    (property "Reference" "Q15" (id 0) (at 101.6 62.23 90))
     (property "Value" "2N3904" (id 1) (at 102.87 59.69 90))
     (property "Footprint" "Package_TO_SOT_THT:TO-92_Inline" (id 2) (at 95.25 67.31 0)
@@
   (symbol (lib_id "Amplifier_Operational:TL074") (at 179.07 81.28 0) (mirror x) (unit 1)
     (in_bom yes) (on_board yes)
-    (property "Reference" "U3" (id 0) (at 179.07 72.39 0))
+    (property "Reference" "U8" (id 0) (at 179.07 72.39 0))
     (property "Value" "TL074" (id 1) (at 179.07 74.93 0))
     (property "Footprint" "Package_SO:SOIC-14_3.9x8.7mm_P1.27mm" (id 2) (at 177.8 83.82 0)
@@
   (symbol (lib_id "Device:LED") (at 217.17 83.82 90) (unit 1)
     (in_bom yes) (on_board yes) (fields_autoplaced)
-    (property "Reference" "D9" (id 0) (at 220.98 84.1374 90)
+    (property "Reference" "D6" (id 0) (at 220.98 84.1374 90)
       (effects (font (size 1.27 1.27)) (justify right))
     )
@@
   (symbol (lib_id "Device:R") (at 133.985 100.33 90) (unit 1)
     (in_bom yes) (on_board yes) (fields_autoplaced)
-    (property "Reference" "R29" (id 0) (at 133.985 93.98 90))
+    (property "Reference" "R41" (id 0) (at 133.985 93.98 90))
     (property "Value" "1M" (id 1) (at 133.985 96.52 90))
     (property "Footprint" "Resistor_THT:R_Axial_DIN0207_L6.3mm_D2.5mm_P7.62mm_Horizontal" (id 2) (at 133.985 102.108 90)
@@
   (symbol (lib_id "Device:R") (at 154.94 62.23 90) (unit 1)
     (in_bom yes) (on_board yes)
-    (property "Reference" "R26" (id 0) (at 154.94 56.515 90))
+    (property "Reference" "R64" (id 0) (at 154.94 56.515 90))
     (property "Value" "100K" (id 1) (at 154.94 58.42 90))
     (property "Footprint" "Resistor_THT:R_Axial_DIN0207_L6.3mm_D2.5mm_P7.62mm_Horizontal" (id 2) (at 154.94 64.008 90)
@@
   (symbol (lib_id "Device:LED") (at 217.17 73.66 90) (unit 1)
     (in_bom yes) (on_board yes) (fields_autoplaced)
-    (property "Reference" "D6" (id 0) (at 220.98 73.9774 90)
+    (property "Reference" "D2" (id 0) (at 220.98 73.9774 90)
       (effects (font (size 1.27 1.27)) (justify right))
     )
@@
   (symbol (lib_id "Device:R") (at 165.1 106.045 0) (unit 1)
     (in_bom yes) (on_board yes) (fields_autoplaced)
-    (property "Reference" "R30" (id 0) (at 167.64 104.7749 0)
-      (effects (font (size 1.27 1.27)) (justify left))
-    )
+    (property "Reference" "R19" (id 0) (at 167.64 104.7749 0)
+      (effects (font (size 1.27 1.27)) (justify left))
+    )
