File: hardware/KiCad/LivSynth_0v1/ModMatrix.kicad_sch (KiCad schematic)
At the start: 7 parts, among them SW3 SW_SP3T, SW4 SW_SP3T, SW5 SW_SPDT

Commit message: Fill all title blocks
Other:
- title: (none) -> LivSynth - ModMatrix
Changed lines of the file:
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@@
   (paper "A4")
   (title_block
+    (title "LivSynth - ModMatrix")
     (date "2022-07-18")
     (rev "${Version}")

Commit message: Initial Routing finished
Parts:
- removed SW3, SW4: SW_SP3T, symbol Switch:SW_SP3T
- added RV22: 100K, SloBlo:Alpha_RD901F, symbol Device:R_Potentiometer
- added SW3: SW_SPDT, SloBlo:SW_Toggle_MS500C, symbol Switch:SW_SPDT
- RV6, RV7, RV8, RV9: footprint (none) -> SloBlo:Alpha_RD901F
- SW5: footprint (none) -> SloBlo:SW_Toggle_MS500C
Connections:
- net EG_IN: now also RV22.3, SW3.1 (A)
- net VGND: now also RV22.1
- net at RV8.3: now also RV9.3, SW5.2 (B), SW3.3 (C)
- net at RV6.3: now also SW3.2 (B)
- net VCF_CV_OUT renamed VCF_LFO_OUT
- new net VCF_EG_OUT: RV22.2
- no-connect marks 2 -> 0
Other:
- moved on the sheet: RV8
Changed lines of the file:
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@@
     (company "SloBlo Labs")
   )
-  (junction (at 153.035 95.885) (diameter 0) (color 0 0 0 0)
-  )
   (junction (at 130.81 90.805) (diameter 0) (color 0 0 0 0)
   )
@@
   (junction (at 130.81 126.365) (diameter 0) (color 0 0 0 0)
   )
-  (no_connect (at 158.115 93.345))
-  (no_connect (at 158.115 67.31))
+  (junction (at 153.035 126.365) (diameter 0) (color 0 0 0 0)
+  )
+  (wire (pts (xy 184.15 126.365) (xy 153.035 126.365))
+    (stroke (width 0) (type default) (color 0 0 0 0))
+  )
   (wire (pts (xy 105.41 90.805) (xy 130.81 90.805))
     (stroke (width 0) (type default) (color 0 0 0 0))
   )
-  (wire (pts (xy 184.15 104.775) (xy 184.15 106.68))
+  (wire (pts (xy 184.15 137.16) (xy 184.15 139.065))
     (stroke (width 0) (type default) (color 0 0 0 0))
   )
@@
     (stroke (width 0) (type default) (color 0 0 0 0))
   )
+  (wire (pts (xy 184.15 102.235) (xy 184.15 104.14))
+    (stroke (width 0) (type default) (color 0 0 0 0))
+  )
   (wire (pts (xy 130.81 90.805) (xy 147.955 90.805))
     (stroke (width 0) (type default) (color 0 0 0 0))
   )
-  (wire (pts (xy 187.96 100.965) (xy 190.5 100.965))
+  (wire (pts (xy 184.15 90.805) (xy 184.15 94.615))
+    (stroke (width 0) (type default) (color 0 0 0 0))
+  )
+  (wire (pts (xy 187.96 133.35) (xy 190.5 133.35))
     (stroke (width 0) (type default) (color 0 0 0 0))
   )
@@
     (stroke (width 0) (type default) (color 0 0 0 0))
   )
-  (wire (pts (xy 179.07 106.68) (xy 184.15 106.68))
+  (wire (pts (xy 179.07 139.065) (xy 184.15 139.065))
     (stroke (width 0) (type default) (color 0 0 0 0))
   )
@@
     (stroke (width 0) (type default) (color 0 0 0 0))
   )
-  (wire (pts (xy 158.115 95.885) (xy 153.035 95.885))
-    (stroke (width 0) (type default) (color 0 0 0 0))
-  )
   (wire (pts (xy 184.15 71.12) (xy 184.15 67.31))
     (stroke (width 0) (type default) (color 0 0 0 0))
@@
     (stroke (width 0) (type default) (color 0 0 0 0))
   )
-  (wire (pts (xy 147.955 90.805) (xy 158.115 90.805))
+  (wire (pts (xy 147.955 90.805) (xy 184.15 90.805))
     (stroke (width 0) (type default) (color 0 0 0 0))
   )
@@
     (stroke (width 0) (type default) (color 0 0 0 0))
   )
-  (wire (pts (xy 168.275 93.345) (xy 184.15 93.345))
-    (stroke (width 0) (type default) (color 0 0 0 0))
-  )
   (wire (pts (xy 125.73 104.14) (xy 130.81 104.14))
     (stroke (width 0) (type default) (color 0 0 0 0))
@@
     (stroke (width 0) (type default) (color 0 0 0 0))
   )
+  (wire (pts (xy 184.15 129.54) (xy 184.15 126.365))
+    (stroke (width 0) (type default) (color 0 0 0 0))
+  )
   (wire (pts (xy 130.81 126.365) (xy 130.81 129.54))
     (stroke (width 0) (type default) (color 0 0 0 0))
@@
     (stroke (width 0) (type default) (color 0 0 0 0))
   )
-  (wire (pts (xy 184.15 93.345) (xy 184.15 97.155))
+  (wire (pts (xy 179.07 104.14) (xy 184.15 104.14))
     (stroke (width 0) (type default) (color 0 0 0 0))
   )
@@
     (stroke (width 0) (type default) (color 0 0 0 0))
   )
-  (wire (pts (xy 153.035 95.885) (xy 153.035 126.365))
-    (stroke (width 0) (type default) (color 0 0 0 0))
-  )
-  (wire (pts (xy 153.035 69.85) (xy 153.035 95.885))
+  (wire (pts (xy 153.035 69.85) (xy 153.035 126.365))
+    (stroke (width 0) (type default) (color 0 0 0 0))
+  )
+  (wire (pts (xy 187.96 98.425) (xy 190.5 98.425))
     (stroke (width 0) (type default) (color 0 0 0 0))
   )
@@
     (effects (font (size 1.27 1.27)) (justify left bottom))
   )
-  (global_label "VGND" (shape input) (at 179.07 106.68 180) (fields_autoplaced)
-    (effects (font (size 1.27 1.27)) (justify right))
-    (property "Intersheet References" "${INTERSHEET_REFS}" (id 0) (at 171.6979 106.6006 0)
+  (global_label "VGND" (shape input) (at 179.07 139.065 180) (fields_autoplaced)
+    (effects (font (size 1.27 1.27)) (justify right))
+    (property "Intersheet References" "${INTERSHEET_REFS}" (id 0) (at 171.6979 138.9856 0)
+      (effects (font (size 1.27 1.27)) (justify right) hide)
+    )
+  )
+  (global_label "VGND" (shape input) (at 179.07 104.14 180) (fields_autoplaced)
+    (effects (font (size 1.27 1.27)) (justify right))
+    (property "Intersheet References" "${INTERSHEET_REFS}" (id 0) (at 171.6979 104.0606 0)
       (effects (font (size 1.27 1.27)) (justify right) hide)
     )
@@
     (effects (font (size 1.27 1.27)) (justify left))
   )
-  (hierarchical_label "VCF_CV_OUT" (shape output) (at 190.5 100.965 0)
+  (hierarchical_label "VCF_LFO_OUT" (shape output) (at 190.5 133.35 0)
     (effects (font (size 1.27 1.27)) (justify left))
   )
@@
     (effects (font (size 1.27 1.27)) (justify right))
   )
+  (hierarchical_label "VCF_EG_OUT" (shape output) (at 190.5 98.425 0)
+    (effects (font (size 1.27 1.27)) (justify left))
+  )
   (hierarchical_label "EG_IN" (shape input) (at 105.41 90.805 180)
     (effects (font (size 1.27 1.27)) (justify right))
   )
-  (symbol (lib_id "Device:R_Potentiometer") (at 184.15 100.965 0) (mirror x) (unit 1)
-    (in_bom yes) (on_board yes) (fields_autoplaced)
-    (property "Reference" "RV8" (id 0) (at 181.61 99.6949 0)
-      (effects (font (size 1.27 1.27)) (justify right))
-    )
-    (property "Value" "100K" (id 1) (at 181.61 102.2349 0)
-      (effects (font (size 1.27 1.27)) (justify right))
-    )
-    (property "Footprint" "" (id 2) (at 184.15 100.965 0)
-      (effects (font (size 1.27 1.27)) hide)
-    )
-    (property "Datasheet" "~" (id 3) (at 184.15 100.965 0)
+  (symbol (lib_id "Device:R_Potentiometer") (at 184.15 98.425 0) (mirror x) (unit 1)
+    (in_bom yes) (on_board yes) (fields_autoplaced)
+    (property "Reference" "RV22" (id 0) (at 181.61 97.1549 0)
+      (effects (font (size 1.27 1.27)) (justify right))
+    )
+    (property "Value" "100K" (id 1) (at 181.61 99.6949 0)
+      (effects (font (size 1.27 1.27)) (justify right))
+    )
+    (property "Footprint" "SloBlo:Alpha_RD901F" (id 2) (at 184.15 98.425 0)
+      (effects (font (size 1.27 1.27)) hide)
+    )
+    (property "Datasheet" "~" (id 3) (at 184.15 98.425 0)
+      (effects (font (size 1.27 1.27)) hide)
+    )
+    (pin "1")
+    (pin "2")
+    (pin "3")
+  )
+  (symbol (lib_id "Device:R_Potentiometer") (at 184.15 133.35 0) (mirror x) (unit 1)
+    (in_bom yes) (on_board yes) (fields_autoplaced)
+    (property "Reference" "RV8" (id 0) (at 181.61 132.0799 0)
+      (effects (font (size 1.27 1.27)) (justify right))
+    )
+    (property "Value" "100K" (id 1) (at 181.61 134.6199 0)
+      (effects (font (size 1.27 1.27)) (justify right))
+    )
+    (property "Footprint" "SloBlo:Alpha_RD901F" (id 2) (at 184.15 133.35 0)
+      (effects (font (size 1.27 1.27)) hide)
+    )
+    (property "Datasheet" "~" (id 3) (at 184.15 133.35 0)
       (effects (font (size 1.27 1.27)) hide)
     )
@@
       (effects (font (size 1.27 1.27)) (justify right))
     )
-    (property "Footprint" "" (id 2) (at 130.81 133.35 0)
+    (property "Footprint" "SloBlo:Alpha_RD901F" (id 2) (at 130.81 133.35 0)
       (effects (font (size 1.27 1.27)) hide)
     )
@@
     (pin "3")
   )
-  (symbol (lib_id "Switch:SW_SP3T") (at 163.195 93.345 0) (mirror y) (unit 1)
-    (in_bom yes) (on_board yes) (fields_autoplaced)
-    (property "Reference" "SW4" (id 0) (at 163.195 85.725 0))
-    (property "Value" "SW_SP3T" (id 1) (at 163.195 88.265 0))
-    (property "Footprint" "" (id 2) (at 179.07 88.9 0)
-      (effects (font (size 1.27 1.27)) hide)
-    )
-    (property "Datasheet" "~" (id 3) (at 179.07 88.9 0)
-      (effects (font (size 1.27 1.27)) hide)
-    )
-    (pin "1")
-    (pin "2")
-    (pin "3")
-    (pin "4")
+  (symbol (lib_id "Switch:SW_SPDT") (at 163.195 67.31 0) (mirror y) (unit 1)
+    (in_bom yes) (on_board yes) (fields_autoplaced)
+    (property "Reference" "SW3" (id 0) (at 163.195 59.69 0))
+    (property "Value" "SW_SPDT" (id 1) (at 163.195 62.23 0))
+    (property "Footprint" "SloBlo:SW_Toggle_MS500C" (id 2) (at 163.195 67.31 0)
+      (effects (font (size 1.27 1.27)) hide)
+    )
+    (property "Datasheet" "~" (id 3) (at 163.195 67.31 0)
+      (effects (font (size 1.27 1.27)) hide)
+    )
+    (pin "1")
+    (pin "2")
+    (pin "3")
   )
   (symbol (lib_id "Device:R_Potentiometer") (at 130.81 98.425 0) (mirror x) (unit 1)
@@
       (effects (font (size 1.27 1.27)) (justify right))
     )
-    (property "Footprint" "" (id 2) (at 130.81 98.425 0)
+    (property "Footprint" "SloBlo:Alpha_RD901F" (id 2) (at 130.81 98.425 0)
       (effects (font (size 1.27 1.27)) hide)
     )
@@
     (pin "3")
   )
-  (symbol (lib_id "Switch:SW_SP3T") (at 163.195 67.31 0) (mirror y) (unit 1)
-    (in_bom yes) (on_board yes) (fields_autoplaced)
-    (property "Reference" "SW3" (id 0) (at 163.195 59.69 0))
-    (property "Value" "SW_SP3T" (id 1) (at 163.195 62.23 0))
-    (property "Footprint" "" (id 2) (at 179.07 62.865 0)
-      (effects (font (size 1.27 1.27)) hide)
-    )
-    (property "Datasheet" "~" (id 3) (at 179.07 62.865 0)
-      (effects (font (size 1.27 1.27)) hide)
-    )
-    (pin "1")
-    (pin "2")
-    (pin "3")
-    (pin "4")
-  )
   (symbol (lib_id "Device:R_Potentiometer") (at 184.15 74.93 0) (mirror x) (unit 1)
     (in_bom yes) (on_board yes) (fields_autoplaced)
@@
       (effects (font (size 1.27 1.27)) (justify right))
     )
-    (property "Footprint" "" (id 2) (at 184.15 74.93 0)
+    (property "Footprint" "SloBlo:Alpha_RD901F" (id 2) (at 184.15 74.93 0)
       (effects (font (size 1.27 1.27)) hide)
     )
@@
     (property "Reference" "SW5" (id 0) (at 114.3 118.745 0))
     (property "Value" "SW_SPDT" (id 1) (at 114.3 121.285 0))
-    (property "Footprint" "" (id 2) (at 114.3 126.365 0)
-      (effects (font (size 1.27 1.27)) hide)
-    )
+    (property "Footprint" "SloBlo:SW_Toggle_MS500C" (id 2) (at 114.3 126.365 0)
+      (effects (font (size 1.27 1.27)) hide)
+    )

Commit message: 0v1 Ready for Production
Parts:
- renumbered RV7 to RV14, RV22 to RV15, RV9 to RV18, RV8 to RV19, RV6 to RV21, SW5 to SW3, SW3 to SW4
Changed lines of the file:
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@@
   (symbol (lib_id "Device:R_Potentiometer") (at 184.15 98.425 0) (mirror x) (unit 1)
     (in_bom yes) (on_board yes) (fields_autoplaced)
-    (property "Reference" "RV22" (id 0) (at 181.61 97.1549 0)
+    (property "Reference" "RV15" (id 0) (at 181.61 97.1549 0)
       (effects (font (size 1.27 1.27)) (justify right))
     )
@@
   (symbol (lib_id "Device:R_Potentiometer") (at 184.15 133.35 0) (mirror x) (unit 1)
     (in_bom yes) (on_board yes) (fields_autoplaced)
-    (property "Reference" "RV8" (id 0) (at 181.61 132.0799 0)
+    (property "Reference" "RV19" (id 0) (at 181.61 132.0799 0)
       (effects (font (size 1.27 1.27)) (justify right))
     )
@@
   (symbol (lib_id "Device:R_Potentiometer") (at 130.81 133.35 0) (mirror x) (unit 1)
     (in_bom yes) (on_board yes) (fields_autoplaced)
-    (property "Reference" "RV9" (id 0) (at 128.27 132.0799 0)
+    (property "Reference" "RV18" (id 0) (at 128.27 132.0799 0)
       (effects (font (size 1.27 1.27)) (justify right))
     )
@@
   (symbol (lib_id "Switch:SW_SPDT") (at 163.195 67.31 0) (mirror y) (unit 1)
     (in_bom yes) (on_board yes) (fields_autoplaced)
-    (property "Reference" "SW3" (id 0) (at 163.195 59.69 0))
+    (property "Reference" "SW4" (id 0) (at 163.195 59.69 0))
     (property "Value" "SW_SPDT" (id 1) (at 163.195 62.23 0))
     (property "Footprint" "SloBlo:SW_Toggle_MS500C" (id 2) (at 163.195 67.31 0)
@@
   (symbol (lib_id "Device:R_Potentiometer") (at 130.81 98.425 0) (mirror x) (unit 1)
     (in_bom yes) (on_board yes) (fields_autoplaced)
-    (property "Reference" "RV7" (id 0) (at 128.27 97.1549 0)
+    (property "Reference" "RV14" (id 0) (at 128.27 97.1549 0)
       (effects (font (size 1.27 1.27)) (justify right))
     )
@@
   (symbol (lib_id "Device:R_Potentiometer") (at 184.15 74.93 0) (mirror x) (unit 1)
     (in_bom yes) (on_board yes) (fields_autoplaced)
-    (property "Reference" "RV6" (id 0) (at 182.245 73.6599 0)
+    (property "Reference" "RV21" (id 0) (at 182.245 73.6599 0)
       (effects (font (size 1.27 1.27)) (justify right))
     )
@@
   (symbol (lib_id "Switch:SW_SPDT") (at 114.3 126.365 0) (mirror y) (unit 1)
     (in_bom yes) (on_board yes) (fields_autoplaced)
-    (property "Reference" "SW5" (id 0) (at 114.3 118.745 0))
+    (property "Reference" "SW3" (id 0) (at 114.3 118.745 0))
     (property "Value" "SW_SPDT" (id 1) (at 114.3 121.285 0))
     (property "Footprint" "SloBlo:SW_Toggle_MS500C" (id 2) (at 114.3 126.365 0)
