File: hardware/KiCad/LivSynth_0v1/Power.kicad_sch (KiCad schematic)
At the start: 33 parts, among them J1 Barrel_Jack_Switch, U1 TL074, U2 TL074, U3 TL074, U4 TL074, U5 TL074, U6 LM13700, U7 TL072, U8 LM1117-3.3

Commit message: Initial Routing finished
Parts:
- removed U7: TL072, symbol Amplifier_Operational:TL072
- added H1, H2, H3, H4: MountingHole, MountingHole:MountingHole_3.2mm_M3, symbol Mechanical:MountingHole
- added NT2: NetTie_2, NetTie:NetTie-2_SMD_Pad2.0mm, symbol Device:NetTie_2
- added R130: 220, Resistor_THT:R_Axial_DIN0207_L6.3mm_D2.5mm_P7.62mm_Horizontal, symbol Device:R
- added SW4: SW_SPDT, Button_Switch_THT:SW_E-Switch_EG1224_SPDT_Angled, symbol Switch:SW_SPDT
- added TP1: VGND, Connector_PinHeader_2.54mm:PinHeader_1x01_P2.54mm_Vertical, symbol Connector:TestPoint
- added unit 2 of U1
- added unit 3 of U1
- added unit 4 of U1
- added unit 1 of U1
- BT1: footprint (none) -> Battery:BatteryHolder_Eagle_12BH611-GR
- FB1: footprint (none) -> Inductor_SMD:L_0603_1608Metric
- J1: footprint (none) -> Connector_BarrelJack:BarrelJack_Wuerth_6941xx301002
- U1, U2, U3, U4, U5: footprint (none) -> Package_SO:SOIC-14_3.9x8.7mm_P1.27mm
- U6: footprint (none) -> Package_SO:SOP-16_3.9x9.9mm_P1.27mm
- U8: footprint (none) -> Package_TO_SOT_SMD:SOT-223
Connections:
- net +9V: now also R130.2, SW4.3 (C); no longer D1.1 (K)
- net GND: now also NT2.1; no longer BT1.2 (-), J1.1
- net VGND: now also TP1.1
- net at C13.1, R1.2, R3.1: now also U1.3 (+), U1.5 (+)
- net at R4.1: now also U1.6 (-), U1.7
- net BAT_P: now reaches BT1.1 (+), J1.3
- net at R2.1: now also U1.1, U1.2 (-)
- new net: D1.1 (K), SW4.2 (B)
- new net BAT_N: BT1.2 (-), J1.1, NT2.2
- new net VBUS: R130.1
- no-connect marks 0 -> 7
Other:
- note added: "Centre negative design: Pin 3 opens when a DC barrel jack is plugged in, disconnecting the battery"
- note added: "Power Switch"
- note removed: "Centre negative design: Pin 3 opens when a DC barrel jack is plugged in disconnecting the battery"
- moved on the sheet: BT1, C14, D1, J1

Commit message: Rework for polyester film capacitors
Parts:
- C1, C10, C11, C12, C2, C3, C4, C5, C6, C7, C8, C9: footprint Capacitor_THT:C_Disc_D3.0mm_W1.6mm_P2.50mm -> Capacitor_THT:C_Rect_L7.2mm_W2.5mm_P5.00mm_FKS2_FKP2_MKS2_MKP2
- C13, C16, C17: footprint Capacitor_THT:C_Disc_D3.0mm_W1.6mm_P2.50mm -> Capacitor_THT:C_Rect_L7.2mm_W5.5mm_P5.00mm_FKS2_FKP2_MKS2_MKP2
- J1: footprint Connector_BarrelJack:BarrelJack_Wuerth_6941xx301002 -> Connector_BarrelJack:BarrelJack_CUI_PJ-102AH_Horizontal
Changed lines of the file:
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@@
       (effects (font (size 1.27 1.27)) (justify left))
     )
-    (property "Footprint" "Capacitor_THT:C_Disc_D3.0mm_W1.6mm_P2.50mm" (id 2) (at 135.255 85.09 0)
+    (property "Footprint" "Capacitor_THT:C_Rect_L7.2mm_W2.5mm_P5.00mm_FKS2_FKP2_MKS2_MKP2" (id 2) (at 135.255 85.09 0)
       (effects (font (size 1.27 1.27)) hide)
     )
@@
       (effects (font (size 1.27 1.27)) (justify left))
     )
-    (property "Footprint" "Capacitor_THT:C_Disc_D3.0mm_W1.6mm_P2.50mm" (id 2) (at 135.255 43.18 0)
+    (property "Footprint" "Capacitor_THT:C_Rect_L7.2mm_W2.5mm_P5.00mm_FKS2_FKP2_MKS2_MKP2" (id 2) (at 135.255 43.18 0)
       (effects (font (size 1.27 1.27)) hide)
     )
@@
       (effects (font (size 1.27 1.27)) (justify right))
     )
-    (property "Footprint" "Connector_BarrelJack:BarrelJack_Wuerth_6941xx301002" (id 2) (at 59.69 42.164 0)
+    (property "Footprint" "Connector_BarrelJack:BarrelJack_CUI_PJ-102AH_Horizontal" (id 2) (at 59.69 42.164 0)
       (effects (font (size 1.27 1.27)) hide)
     )
@@
       (effects (font (size 1.27 1.27)) (justify left))
     )
-    (property "Footprint" "Capacitor_THT:C_Disc_D3.0mm_W1.6mm_P2.50mm" (id 2) (at 198.12 32.385 0)
+    (property "Footprint" "Capacitor_THT:C_Rect_L7.2mm_W2.5mm_P5.00mm_FKS2_FKP2_MKS2_MKP2" (id 2) (at 198.12 32.385 0)
       (effects (font (size 1.27 1.27)) hide)
     )
@@
       (effects (font (size 1.27 1.27)) (justify left))
     )
-    (property "Footprint" "Capacitor_THT:C_Disc_D3.0mm_W1.6mm_P2.50mm" (id 2) (at 198.12 43.18 0)
+    (property "Footprint" "Capacitor_THT:C_Rect_L7.2mm_W2.5mm_P5.00mm_FKS2_FKP2_MKS2_MKP2" (id 2) (at 198.12 43.18 0)
       (effects (font (size 1.27 1.27)) hide)
     )
@@
       (effects (font (size 1.27 1.27)) (justify left))
     )
-    (property "Footprint" "Capacitor_THT:C_Disc_D3.0mm_W1.6mm_P2.50mm" (id 2) (at 135.255 32.385 0)
+    (property "Footprint" "Capacitor_THT:C_Rect_L7.2mm_W2.5mm_P5.00mm_FKS2_FKP2_MKS2_MKP2" (id 2) (at 135.255 32.385 0)
       (effects (font (size 1.27 1.27)) hide)
     )
@@
       (effects (font (size 1.27 1.27)) (justify left))
     )
-    (property "Footprint" "Capacitor_THT:C_Disc_D3.0mm_W1.6mm_P2.50mm" (id 2) (at 73.66 173.99 0)
+    (property "Footprint" "Capacitor_THT:C_Rect_L7.2mm_W5.5mm_P5.00mm_FKS2_FKP2_MKS2_MKP2" (id 2) (at 73.66 173.99 0)
       (effects (font (size 1.27 1.27)) hide)
     )
@@
       (effects (font (size 1.27 1.27)) (justify left))
     )
-    (property "Footprint" "Capacitor_THT:C_Disc_D3.0mm_W1.6mm_P2.50mm" (id 2) (at 219.075 43.18 0)
+    (property "Footprint" "Capacitor_THT:C_Rect_L7.2mm_W2.5mm_P5.00mm_FKS2_FKP2_MKS2_MKP2" (id 2) (at 219.075 43.18 0)
       (effects (font (size 1.27 1.27)) hide)
     )
@@
       (effects (font (size 1.27 1.27)) (justify left))
     )
-    (property "Footprint" "Capacitor_THT:C_Disc_D3.0mm_W1.6mm_P2.50mm" (id 2) (at 156.21 32.385 0)
+    (property "Footprint" "Capacitor_THT:C_Rect_L7.2mm_W2.5mm_P5.00mm_FKS2_FKP2_MKS2_MKP2" (id 2) (at 156.21 32.385 0)
       (effects (font (size 1.27 1.27)) hide)
     )
@@
       (effects (font (size 1.27 1.27)) (justify left))
     )
-    (property "Footprint" "Capacitor_THT:C_Disc_D3.0mm_W1.6mm_P2.50mm" (id 2) (at 219.075 32.385 0)
+    (property "Footprint" "Capacitor_THT:C_Rect_L7.2mm_W2.5mm_P5.00mm_FKS2_FKP2_MKS2_MKP2" (id 2) (at 219.075 32.385 0)
       (effects (font (size 1.27 1.27)) hide)
     )
@@
       (effects (font (size 1.27 1.27)) (justify left))
     )
-    (property "Footprint" "Capacitor_THT:C_Disc_D3.0mm_W1.6mm_P2.50mm" (id 2) (at 177.165 32.385 0)
+    (property "Footprint" "Capacitor_THT:C_Rect_L7.2mm_W2.5mm_P5.00mm_FKS2_FKP2_MKS2_MKP2" (id 2) (at 177.165 32.385 0)
       (effects (font (size 1.27 1.27)) hide)
     )
@@
       (effects (font (size 1.27 1.27)) (justify left))
     )
-    (property "Footprint" "Capacitor_THT:C_Disc_D3.0mm_W1.6mm_P2.50mm" (id 2) (at 177.165 43.18 0)
+    (property "Footprint" "Capacitor_THT:C_Rect_L7.2mm_W2.5mm_P5.00mm_FKS2_FKP2_MKS2_MKP2" (id 2) (at 177.165 43.18 0)
       (effects (font (size 1.27 1.27)) hide)
     )
@@
       (effects (font (size 1.27 1.27)) (justify left))
     )
-    (property "Footprint" "Capacitor_THT:C_Disc_D3.0mm_W1.6mm_P2.50mm" (id 2) (at 156.21 43.18 0)
+    (property "Footprint" "Capacitor_THT:C_Rect_L7.2mm_W2.5mm_P5.00mm_FKS2_FKP2_MKS2_MKP2" (id 2) (at 156.21 43.18 0)
       (effects (font (size 1.27 1.27)) hide)
     )
@@
       (effects (font (size 1.27 1.27)) (justify left))
     )
-    (property "Footprint" "Capacitor_THT:C_Disc_D3.0mm_W1.6mm_P2.50mm" (id 2) (at 135.255 74.295 0)
+    (property "Footprint" "Capacitor_THT:C_Rect_L7.2mm_W2.5mm_P5.00mm_FKS2_FKP2_MKS2_MKP2" (id 2) (at 135.255 74.295 0)
       (effects (font (size 1.27 1.27)) hide)
     )
@@
       (effects (font (size 1.27 1.27)) (justify left))
     )
-    (property "Footprint" "Capacitor_THT:C_Disc_D3.0mm_W1.6mm_P2.50mm" (id 2) (at 43.815 173.99 0)
+    (property "Footprint" "Capacitor_THT:C_Rect_L7.2mm_W5.5mm_P5.00mm_FKS2_FKP2_MKS2_MKP2" (id 2) (at 43.815 173.99 0)
       (effects (font (size 1.27 1.27)) hide)
     )
@@
       (effects (font (size 1.27 1.27)) (justify left))
     )
-    (property "Footprint" "Capacitor_THT:C_Disc_D3.0mm_W1.6mm_P2.50mm" (id 2) (at 43.5102 98.425 0)
-      (effects (font (size 1.27 1.27)) hide)
-    )
+    (property "Footprint" "Capacitor_THT:C_Rect_L7.2mm_W5.5mm_P5.00mm_FKS2_FKP2_MKS2_MKP2" (id 2) (at 43.5102 98.425 0)
+      (effects (font (size 1.27 1.27)) hide)
+    )

Commit message: Use correct Elko sizes (8mm/3.5mm)
Parts:
- C14, C15: footprint Capacitor_THT:CP_Radial_D8.0mm_P5.00mm -> Capacitor_THT:CP_Radial_D8.0mm_P3.50mm
Changed lines of the file:
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@@
       (effects (font (size 1.27 1.27)) (justify left))
     )
-    (property "Footprint" "Capacitor_THT:CP_Radial_D8.0mm_P5.00mm" (id 2) (at 74.6252 149.86 0)
+    (property "Footprint" "Capacitor_THT:CP_Radial_D8.0mm_P3.50mm" (id 2) (at 74.6252 149.86 0)
       (effects (font (size 1.27 1.27)) hide)
     )
@@
       (effects (font (size 1.27 1.27)) (justify left))
     )
-    (property "Footprint" "Capacitor_THT:CP_Radial_D8.0mm_P5.00mm" (id 2) (at 45.4152 149.86 0)
-      (effects (font (size 1.27 1.27)) hide)
-    )
+    (property "Footprint" "Capacitor_THT:CP_Radial_D8.0mm_P3.50mm" (id 2) (at 45.4152 149.86 0)
+      (effects (font (size 1.27 1.27)) hide)
+    )

Commit message: 0v1 Ready for Production
Parts:
- renumbered C13 to C1, C2 to C10, C5 to C12, C4 to C15, C9 to C18, C14 to C20, C7 to C24, C3 to C25, C11 to C28, C10 to C29, C6 to C3, C15 to C31, C17 to C34, C16 to C35, C8 to C39, C1 to C4, C12 to C41, J1 to J5, R4 to R1, R3 to R11, R1 to R12, R130 to R56, SW4 to SW6, U2 to U3, U8 to U5, U5 to U6, U6 to U7, U3 to U8
Changed lines of the file:
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@@
   (symbol (lib_id "Device:C_Small") (at 135.255 85.09 0) (unit 1)
     (in_bom yes) (on_board yes) (fields_autoplaced)
-    (property "Reference" "C12" (id 0) (at 137.795 83.8262 0)
+    (property "Reference" "C41" (id 0) (at 137.795 83.8262 0)
       (effects (font (size 1.27 1.27)) (justify left))
     )
@@
   (symbol (lib_id "Device:C_Polarized") (at 73.66 146.05 0) (unit 1)
     (in_bom yes) (on_board yes) (fields_autoplaced)
-    (property "Reference" "C15" (id 0) (at 77.47 143.8909 0)
+    (property "Reference" "C31" (id 0) (at 77.47 143.8909 0)
       (effects (font (size 1.27 1.27)) (justify left))
     )
@@
   (symbol (lib_id "Amplifier_Operational:TL074") (at 211.455 38.1 0) (unit 5)
     (in_bom yes) (on_board yes) (fields_autoplaced)
-    (property "Reference" "U5" (id 0) (at 210.185 36.8299 0)
+    (property "Reference" "U6" (id 0) (at 210.185 36.8299 0)
       (effects (font (size 1.27 1.27)) (justify left))
     )
@@
   (symbol (lib_id "Regulator_Linear:LM1117-3.3") (at 59.055 140.97 0) (unit 1)
     (in_bom yes) (on_board yes) (fields_autoplaced)
-    (property "Reference" "U8" (id 0) (at 59.055 133.35 0))
+    (property "Reference" "U5" (id 0) (at 59.055 133.35 0))
     (property "Value" "LM1117-3.3" (id 1) (at 59.055 135.89 0))
     (property "Footprint" "Package_TO_SOT_SMD:SOT-223" (id 2) (at 59.055 140.97 0)
@@
   (symbol (lib_id "Amplifier_Operational:LM13700") (at 127 79.375 0) (unit 5)
     (in_bom yes) (on_board yes) (fields_autoplaced)
-    (property "Reference" "U6" (id 0) (at 125.095 78.1049 0)
+    (property "Reference" "U7" (id 0) (at 125.095 78.1049 0)
       (effects (font (size 1.27 1.27)) (justify left))
     )
@@
   (symbol (lib_id "Device:C_Small") (at 135.255 43.18 0) (unit 1)
     (in_bom yes) (on_board yes) (fields_autoplaced)
-    (property "Reference" "C6" (id 0) (at 137.795 41.9162 0)
+    (property "Reference" "C3" (id 0) (at 137.795 41.9162 0)
       (effects (font (size 1.27 1.27)) (justify left))
     )
@@
   (symbol (lib_id "Connector:Barrel_Jack_Switch") (at 58.42 43.18 0) (mirror x) (unit 1)
     (in_bom yes) (on_board yes) (fields_autoplaced)
-    (property "Reference" "J1" (id 0) (at 51.435 41.9099 0)
+    (property "Reference" "J5" (id 0) (at 51.435 41.9099 0)
       (effects (font (size 1.27 1.27)) (justify right))
     )
@@
   (symbol (lib_id "Device:R") (at 74.93 111.76 90) (unit 1)
     (in_bom yes) (on_board yes) (fields_autoplaced)
-    (property "Reference" "R4" (id 0) (at 74.93 106.045 90))
+    (property "Reference" "R1" (id 0) (at 74.93 106.045 90))
     (property "Value" "10R" (id 1) (at 74.93 108.585 90))
     (property "Footprint" "Resistor_THT:R_Axial_DIN0207_L6.3mm_D2.5mm_P7.62mm_Horizontal" (id 2) (at 74.93 113.538 90)
@@
   (symbol (lib_id "Device:R") (at 33.655 94.615 0) (unit 1)
     (in_bom yes) (on_board yes) (fields_autoplaced)
-    (property "Reference" "R3" (id 0) (at 36.195 93.3449 0)
+    (property "Reference" "R11" (id 0) (at 36.195 93.3449 0)
       (effects (font (size 1.27 1.27)) (justify left))
     )
@@
   (symbol (lib_id "Device:C_Small") (at 198.12 32.385 0) (unit 1)
     (in_bom yes) (on_board yes) (fields_autoplaced)
-    (property "Reference" "C4" (id 0) (at 200.66 31.1212 0)
+    (property "Reference" "C15" (id 0) (at 200.66 31.1212 0)
       (effects (font (size 1.27 1.27)) (justify left))
     )
@@
   (symbol (lib_id "Device:C_Small") (at 198.12 43.18 0) (unit 1)
     (in_bom yes) (on_board yes) (fields_autoplaced)
-    (property "Reference" "C9" (id 0) (at 200.66 41.9162 0)
+    (property "Reference" "C18" (id 0) (at 200.66 41.9162 0)
       (effects (font (size 1.27 1.27)) (justify left))
     )
@@
   (symbol (lib_id "Device:C_Small") (at 135.255 32.385 0) (unit 1)
     (in_bom yes) (on_board yes) (fields_autoplaced)
-    (property "Reference" "C1" (id 0) (at 137.795 31.1212 0)
+    (property "Reference" "C4" (id 0) (at 137.795 31.1212 0)
       (effects (font (size 1.27 1.27)) (justify left))
     )
@@
   (symbol (lib_id "Device:C_Small") (at 73.66 173.99 0) (mirror y) (unit 1)
     (in_bom yes) (on_board yes) (fields_autoplaced)
-    (property "Reference" "C17" (id 0) (at 70.485 172.7262 0)
+    (property "Reference" "C34" (id 0) (at 70.485 172.7262 0)
       (effects (font (size 1.27 1.27)) (justify left))
     )
@@
   (symbol (lib_id "Device:C_Small") (at 219.075 43.18 0) (unit 1)
     (in_bom yes) (on_board yes) (fields_autoplaced)
-    (property "Reference" "C10" (id 0) (at 221.615 41.9162 0)
+    (property "Reference" "C29" (id 0) (at 221.615 41.9162 0)
       (effects (font (size 1.27 1.27)) (justify left))
     )
@@
   (symbol (lib_id "Device:C_Small") (at 156.21 32.385 0) (unit 1)
     (in_bom yes) (on_board yes) (fields_autoplaced)
-    (property "Reference" "C2" (id 0) (at 158.75 31.1212 0)
+    (property "Reference" "C10" (id 0) (at 158.75 31.1212 0)
       (effects (font (size 1.27 1.27)) (justify left))
     )
@@
   (symbol (lib_id "Device:C_Small") (at 219.075 32.385 0) (unit 1)
     (in_bom yes) (on_board yes) (fields_autoplaced)
-    (property "Reference" "C5" (id 0) (at 221.615 31.1212 0)
+    (property "Reference" "C12" (id 0) (at 221.615 31.1212 0)
       (effects (font (size 1.27 1.27)) (justify left))
     )
@@
   (symbol (lib_id "Amplifier_Operational:TL074") (at 148.59 38.1 0) (unit 5)
     (in_bom yes) (on_board yes) (fields_autoplaced)
-    (property "Reference" "U2" (id 0) (at 147.32 36.8299 0)
+    (property "Reference" "U3" (id 0) (at 147.32 36.8299 0)
       (effects (font (size 1.27 1.27)) (justify left))
     )
@@
   (symbol (lib_id "Device:C_Small") (at 177.165 32.385 0) (unit 1)
     (in_bom yes) (on_board yes) (fields_autoplaced)
-    (property "Reference" "C3" (id 0) (at 179.705 31.1212 0)
+    (property "Reference" "C25" (id 0) (at 179.705 31.1212 0)
       (effects (font (size 1.27 1.27)) (justify left))
     )
@@
   (symbol (lib_id "Device:C_Small") (at 177.165 43.18 0) (unit 1)
     (in_bom yes) (on_board yes) (fields_autoplaced)
-    (property "Reference" "C8" (id 0) (at 179.705 41.9162 0)
+    (property "Reference" "C39" (id 0) (at 179.705 41.9162 0)
       (effects (font (size 1.27 1.27)) (justify left))
     )
@@
   (symbol (lib_id "Device:C_Small") (at 156.21 43.18 0) (unit 1)
     (in_bom yes) (on_board yes) (fields_autoplaced)
-    (property "Reference" "C7" (id 0) (at 158.75 41.9162 0)
+    (property "Reference" "C24" (id 0) (at 158.75 41.9162 0)
       (effects (font (size 1.27 1.27)) (justify left))
     )
@@
   (symbol (lib_id "Device:C_Small") (at 135.255 74.295 0) (unit 1)
     (in_bom yes) (on_board yes) (fields_autoplaced)
-    (property "Reference" "C11" (id 0) (at 137.795 73.0312 0)
+    (property "Reference" "C28" (id 0) (at 137.795 73.0312 0)
       (effects (font (size 1.27 1.27)) (justify left))
     )
@@
   (symbol (lib_id "Device:C_Small") (at 43.815 173.99 0) (mirror y) (unit 1)
     (in_bom yes) (on_board yes) (fields_autoplaced)
-    (property "Reference" "C16" (id 0) (at 40.64 172.7262 0)
+    (property "Reference" "C35" (id 0) (at 40.64 172.7262 0)
       (effects (font (size 1.27 1.27)) (justify left))
     )
@@
   (symbol (lib_id "Device:R") (at 33.655 81.28 0) (unit 1)
     (in_bom yes) (on_board yes) (fields_autoplaced)
-    (property "Reference" "R1" (id 0) (at 36.195 80.0099 0)
+    (property "Reference" "R12" (id 0) (at 36.195 80.0099 0)
       (effects (font (size 1.27 1.27)) (justify left))
     )
@@
   (symbol (lib_id "Device:C") (at 42.545 94.615 0) (unit 1)
     (in_bom yes) (on_board yes) (fields_autoplaced)
-    (property "Reference" "C13" (id 0) (at 45.72 93.3449 0)
+    (property "Reference" "C1" (id 0) (at 45.72 93.3449 0)
       (effects (font (size 1.27 1.27)) (justify left))
     )
@@
   (symbol (lib_id "Device:C_Polarized") (at 44.45 146.05 0) (unit 1)
     (in_bom yes) (on_board yes) (fields_autoplaced)
-    (property "Reference" "C14" (id 0) (at 47.625 143.8909 0)
+    (property "Reference" "C20" (id 0) (at 47.625 143.8909 0)
       (effects (font (size 1.27 1.27)) (justify left))
     )
@@
   (symbol (lib_id "Device:R") (at 38.1 140.97 90) (unit 1)
     (in_bom yes) (on_board yes) (fields_autoplaced)
-    (property "Reference" "R130" (id 0) (at 38.1 134.62 90))
+    (property "Reference" "R56" (id 0) (at 38.1 134.62 90))
     (property "Value" "220" (id 1) (at 38.1 137.16 90))
     (property "Footprint" "Resistor_THT:R_Axial_DIN0207_L6.3mm_D2.5mm_P7.62mm_Horizontal" (id 2) (at 38.1 142.748 90)
@@
   (symbol (lib_id "Switch:SW_SPDT") (at 86.36 40.64 0) (unit 1)
     (in_bom yes) (on_board yes) (fields_autoplaced)
-    (property "Reference" "SW4" (id 0) (at 86.36 33.02 0))
+    (property "Reference" "SW6" (id 0) (at 86.36 33.02 0))
     (property "Value" "SW_SPDT" (id 1) (at 86.36 35.56 0))
     (property "Footprint" "Button_Switch_THT:SW_E-Switch_EG1224_SPDT_Angled" (id 2) (at 86.36 40.64 0)
@@
   (symbol (lib_id "Amplifier_Operational:TL074") (at 169.545 38.1 0) (unit 5)
     (in_bom yes) (on_board yes) (fields_autoplaced)
-    (property "Reference" "U3" (id 0) (at 168.275 36.8299 0)
-      (effects (font (size 1.27 1.27)) (justify left))
-    )
+    (property "Reference" "U8" (id 0) (at 168.275 36.8299 0)
+      (effects (font (size 1.27 1.27)) (justify left))
+    )
