File: hardware/KiCad/LivSynth_0v1/Slew.kicad_sch (KiCad schematic)
At the start: 8 parts, among them J4 Jumper, U1 TL074

Commit message: Fill all title blocks
Other:
- title: (none) -> LivSynth - Slew
Changed lines of the file:
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@@
   (paper "A4")
   (title_block
+    (title "LivSynth - Slew")
     (date "2022-07-18")
     (rev "${Version}")

Commit message: Initial Routing finished
Parts:
- RV1: footprint (none) -> SloBlo:Alpha_RD901F
- U3: renamed from U1; footprint (none) -> Package_SO:SOIC-14_3.9x8.7mm_P1.27mm
Connections:
- net V/OCT_OUT: now also U3.13 (-), U3.14; no longer U3.6 (-), U3.7
- net at C31.1, RV1.2, RV1.3: now also U3.12 (+); no longer U3.5 (+)
- net at R8.2, R9.2: now also U3.5 (+); no longer U3.3 (+)
- net at R6.2, RV1.1: now also U3.7; no longer U3.1
- net at R6.1, R7.2: now also U3.6 (-); no longer U3.2 (-)
Changed lines of the file:
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@@
     (pin "2")
   )
-  (symbol (lib_id "Amplifier_Operational:TL074") (at 161.29 95.885 0) (mirror x) (unit 1)
+  (symbol (lib_id "Amplifier_Operational:TL074") (at 161.29 95.885 0) (mirror x) (unit 2)
     (in_bom yes) (on_board yes)
-    (property "Reference" "U1" (id 0) (at 161.29 88.265 0))
+    (property "Reference" "U3" (id 0) (at 161.29 88.265 0))
     (property "Value" "TL074" (id 1) (at 161.29 90.17 0))
-    (property "Footprint" "" (id 2) (at 160.02 98.425 0)
+    (property "Footprint" "Package_SO:SOIC-14_3.9x8.7mm_P1.27mm" (id 2) (at 160.02 98.425 0)
       (effects (font (size 1.27 1.27)) hide)
     )
@@
     (property "Reference" "RV1" (id 0) (at 181.61 99.695 90))
     (property "Value" "100K" (id 1) (at 181.61 102.235 90))
-    (property "Footprint" "" (id 2) (at 181.61 95.885 0)
+    (property "Footprint" "SloBlo:Alpha_RD901F" (id 2) (at 181.61 95.885 0)
       (effects (font (size 1.27 1.27)) hide)
     )
@@
     (pin "2")
   )
-  (symbol (lib_id "Amplifier_Operational:TL074") (at 212.725 93.345 0) (mirror x) (unit 2)
+  (symbol (lib_id "Amplifier_Operational:TL074") (at 212.725 93.345 0) (mirror x) (unit 4)
     (in_bom yes) (on_board yes)
-    (property "Reference" "U1" (id 0) (at 212.725 85.725 0))
+    (property "Reference" "U3" (id 0) (at 212.725 85.725 0))
     (property "Value" "TL074" (id 1) (at 212.725 87.63 0))
-    (property "Footprint" "" (id 2) (at 211.455 95.885 0)
+    (property "Footprint" "Package_SO:SOIC-14_3.9x8.7mm_P1.27mm" (id 2) (at 211.455 95.885 0)
       (effects (font (size 1.27 1.27)) hide)
     )

Commit message: Rework for polyester film capacitors
Parts:
- C31: footprint Capacitor_THT:C_Disc_D3.0mm_W1.6mm_P2.50mm -> Capacitor_THT:C_Rect_L7.2mm_W2.5mm_P5.00mm_FKS2_FKP2_MKS2_MKP2
Changed lines of the file:
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@@
       (effects (font (size 1.27 1.27)) (justify left))
     )
-    (property "Footprint" "Capacitor_THT:C_Disc_D3.0mm_W1.6mm_P2.50mm" (id 2) (at 197.8152 106.045 0)
+    (property "Footprint" "Capacitor_THT:C_Rect_L7.2mm_W2.5mm_P5.00mm_FKS2_FKP2_MKS2_MKP2" (id 2) (at 197.8152 106.045 0)
       (effects (font (size 1.27 1.27)) hide)
     )

Commit message: 0v1 Ready for Production
Parts:
- renumbered C31 to C40, J4 to J17, R8 to R83, R7 to R84, R9 to R85, R6 to R86, RV1 to RV20, U3 to U8
Changed lines of the file:
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@@
   (symbol (lib_id "Device:C") (at 196.85 102.235 0) (unit 1)
     (in_bom yes) (on_board yes) (fields_autoplaced)
-    (property "Reference" "C31" (id 0) (at 200.66 100.9649 0)
+    (property "Reference" "C40" (id 0) (at 200.66 100.9649 0)
       (effects (font (size 1.27 1.27)) (justify left))
     )
@@
   (symbol (lib_id "Device:R") (at 144.78 98.425 90) (unit 1)
     (in_bom yes) (on_board yes)
-    (property "Reference" "R8" (id 0) (at 144.78 102.87 90))
+    (property "Reference" "R83" (id 0) (at 144.78 102.87 90))
     (property "Value" "100K" (id 1) (at 144.78 100.965 90))
     (property "Footprint" "Resistor_THT:R_Axial_DIN0207_L6.3mm_D2.5mm_P7.62mm_Horizontal" (id 2) (at 144.78 100.203 90)
@@
   (symbol (lib_id "Amplifier_Operational:TL074") (at 161.29 95.885 0) (mirror x) (unit 2)
     (in_bom yes) (on_board yes)
-    (property "Reference" "U3" (id 0) (at 161.29 88.265 0))
+    (property "Reference" "U8" (id 0) (at 161.29 88.265 0))
     (property "Value" "TL074" (id 1) (at 161.29 90.17 0))
     (property "Footprint" "Package_SO:SOIC-14_3.9x8.7mm_P1.27mm" (id 2) (at 160.02 98.425 0)
@@
   (symbol (lib_id "Device:R_Potentiometer") (at 181.61 95.885 90) (unit 1)
     (in_bom yes) (on_board yes) (fields_autoplaced)
-    (property "Reference" "RV1" (id 0) (at 181.61 99.695 90))
+    (property "Reference" "RV20" (id 0) (at 181.61 99.695 90))
     (property "Value" "100K" (id 1) (at 181.61 102.235 90))
     (property "Footprint" "SloBlo:Alpha_RD901F" (id 2) (at 181.61 95.885 0)
@@
   (symbol (lib_id "Device:R") (at 161.925 82.55 90) (unit 1)
     (in_bom yes) (on_board yes)
-    (property "Reference" "R6" (id 0) (at 161.925 78.105 90))
+    (property "Reference" "R86" (id 0) (at 161.925 78.105 90))
     (property "Value" "100K" (id 1) (at 161.925 80.01 90))
     (property "Footprint" "Resistor_THT:R_Axial_DIN0207_L6.3mm_D2.5mm_P7.62mm_Horizontal" (id 2) (at 161.925 84.328 90)
@@
   (symbol (lib_id "Connector:Conn_01x02_Male") (at 121.285 93.345 90) (mirror x) (unit 1)
     (in_bom yes) (on_board yes) (fields_autoplaced)
-    (property "Reference" "J4" (id 0) (at 125.73 92.7099 90)
+    (property "Reference" "J17" (id 0) (at 125.73 92.7099 90)
       (effects (font (size 1.27 1.27)) (justify right))
     )
@@
   (symbol (lib_id "Amplifier_Operational:TL074") (at 212.725 93.345 0) (mirror x) (unit 4)
     (in_bom yes) (on_board yes)
-    (property "Reference" "U3" (id 0) (at 212.725 85.725 0))
+    (property "Reference" "U8" (id 0) (at 212.725 85.725 0))
     (property "Value" "TL074" (id 1) (at 212.725 87.63 0))
     (property "Footprint" "Package_SO:SOIC-14_3.9x8.7mm_P1.27mm" (id 2) (at 211.455 95.885 0)
@@
   (symbol (lib_id "Device:R") (at 144.78 93.345 90) (unit 1)
     (in_bom yes) (on_board yes)
-    (property "Reference" "R7" (id 0) (at 144.78 88.9 90))
+    (property "Reference" "R84" (id 0) (at 144.78 88.9 90))
     (property "Value" "100K" (id 1) (at 144.78 90.805 90))
     (property "Footprint" "Resistor_THT:R_Axial_DIN0207_L6.3mm_D2.5mm_P7.62mm_Horizontal" (id 2) (at 144.78 95.123 90)
@@
   (symbol (lib_id "Device:R") (at 151.765 106.045 180) (unit 1)
     (in_bom yes) (on_board yes)
-    (property "Reference" "R9" (id 0) (at 147.32 106.045 90))
+    (property "Reference" "R85" (id 0) (at 147.32 106.045 90))
     (property "Value" "340K" (id 1) (at 149.225 106.045 90))
     (property "Footprint" "Resistor_THT:R_Axial_DIN0207_L6.3mm_D2.5mm_P7.62mm_Horizontal" (id 2) (at 153.543 106.045 90)
