File: hardware/KiCad/LivSynth_0v1/VCA.kicad_sch (KiCad schematic)
At the start: 25 parts, among them J11 Jumper, J12 Jumper, Q13 2N3904, Q14 2N3904, U14 TL074, U15 TL074

Commit message: Initial Routing finished
Parts:
- RV17: footprint (none) -> Potentiometer_THT:Potentiometer_Bourns_3296W_Vertical
- RV18: footprint (none) -> SloBlo:Alpha_RD901F
- U2: renamed from U14; footprint (none) -> Package_SO:SOIC-14_3.9x8.7mm_P1.27mm
- U2: renamed from U15; footprint (none) -> Package_SO:SOIC-14_3.9x8.7mm_P1.27mm
Connections:
- net at R63.1, R67.1: now also U2.7; no longer U2.1
- net at R63.2, R66.2: now also U2.6 (-); no longer U2.2 (-)
- net at R68.2, R69.2: now also U2.5 (+); no longer U2.3 (+)
Changed lines of the file:
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@@
     (pin "3")
   )
-  (symbol (lib_id "Amplifier_Operational:TL074") (at 189.865 66.04 0) (mirror x) (unit 1)
+  (symbol (lib_id "Amplifier_Operational:TL074") (at 189.865 66.04 0) (mirror x) (unit 2)
     (in_bom yes) (on_board yes)
-    (property "Reference" "U14" (id 0) (at 189.865 57.15 0))
+    (property "Reference" "U2" (id 0) (at 189.865 57.15 0))
     (property "Value" "TL074" (id 1) (at 189.865 59.69 0))
-    (property "Footprint" "" (id 2) (at 188.595 68.58 0)
+    (property "Footprint" "Package_SO:SOIC-14_3.9x8.7mm_P1.27mm" (id 2) (at 188.595 68.58 0)
       (effects (font (size 1.27 1.27)) hide)
     )
@@
       (effects (font (size 1.27 1.27)) (justify right))
     )
-    (property "Footprint" "" (id 2) (at 76.835 147.32 0)
+    (property "Footprint" "SloBlo:Alpha_RD901F" (id 2) (at 76.835 147.32 0)
       (effects (font (size 1.27 1.27)) hide)
     )
@@
     (property "Reference" "RV17" (id 0) (at 168.275 100.33 90))
     (property "Value" "100K" (id 1) (at 168.275 102.87 90))
-    (property "Footprint" "" (id 2) (at 168.275 97.155 0)
+    (property "Footprint" "Potentiometer_THT:Potentiometer_Bourns_3296W_Vertical" (id 2) (at 168.275 97.155 0)
       (effects (font (size 1.27 1.27)) hide)
     )
@@
   (symbol (lib_id "Amplifier_Operational:TL074") (at 109.855 149.86 0) (mirror x) (unit 1)
     (in_bom yes) (on_board yes)
-    (property "Reference" "U15" (id 0) (at 109.855 140.97 0))
+    (property "Reference" "U2" (id 0) (at 109.855 140.97 0))
     (property "Value" "TL074" (id 1) (at 109.855 143.51 0))
-    (property "Footprint" "" (id 2) (at 108.585 152.4 0)
-      (effects (font (size 1.27 1.27)) hide)
-    )
+    (property "Footprint" "Package_SO:SOIC-14_3.9x8.7mm_P1.27mm" (id 2) (at 108.585 152.4 0)
+      (effects (font (size 1.27 1.27)) hide)
+    )

Commit message: Rework for polyester film capacitors
Parts:
- RV17: footprint Potentiometer_THT:Potentiometer_Bourns_3296W_Vertical -> SloBlo:Potentiometer_Bourns_3296W_Vertical
Changed lines of the file:
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@@
     (property "Reference" "RV17" (id 0) (at 168.275 100.33 90))
     (property "Value" "100K" (id 1) (at 168.275 102.87 90))
-    (property "Footprint" "Potentiometer_THT:Potentiometer_Bourns_3296W_Vertical" (id 2) (at 168.275 97.155 0)
+    (property "Footprint" "SloBlo:Potentiometer_Bourns_3296W_Vertical" (id 2) (at 168.275 97.155 0)
       (effects (font (size 1.27 1.27)) hide)
     )

Commit message: 0v1 Ready for Production
Parts:
- renumbered J12 to J18, J11 to J6, Q13 to Q5, Q14 to Q6, R65 to R17, R72 to R18, R64 to R20, R70 to R3, R67 to R35, R71 to R36, R74 to R37, R73 to R38, R78 to R39, R79 to R57, R76 to R58, R69 to R60, R75 to R62, R77 to R63, R68 to R65, R63 to R66, R66 to R67, RV17 to RV10, RV18 to RV11, U2 to U3
Changed lines of the file:
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@@
   (symbol (lib_id "Device:R") (at 132.08 56.515 0) (unit 1)
     (in_bom yes) (on_board yes)
-    (property "Reference" "R65" (id 0) (at 133.985 55.2449 0)
+    (property "Reference" "R17" (id 0) (at 133.985 55.2449 0)
       (effects (font (size 1.27 1.27)) (justify left))
     )
@@
   (symbol (lib_id "Device:R") (at 120.65 109.22 0) (unit 1)
     (in_bom yes) (on_board yes) (fields_autoplaced)
-    (property "Reference" "R74" (id 0) (at 123.19 107.9499 0)
+    (property "Reference" "R37" (id 0) (at 123.19 107.9499 0)
       (effects (font (size 1.27 1.27)) (justify left))
     )
@@
   (symbol (lib_id "Device:R") (at 95.885 87.63 0) (unit 1)
     (in_bom yes) (on_board yes) (fields_autoplaced)
-    (property "Reference" "R73" (id 0) (at 98.425 86.3599 0)
+    (property "Reference" "R38" (id 0) (at 98.425 86.3599 0)
       (effects (font (size 1.27 1.27)) (justify left))
     )
@@
   (symbol (lib_id "Device:R") (at 86.995 147.32 90) (unit 1)
     (in_bom yes) (on_board yes)
-    (property "Reference" "R78" (id 0) (at 86.995 140.97 90))
+    (property "Reference" "R39" (id 0) (at 86.995 140.97 90))
     (property "Value" "100K" (id 1) (at 86.995 143.51 90))
     (property "Footprint" "Resistor_THT:R_Axial_DIN0207_L6.3mm_D2.5mm_P7.62mm_Horizontal" (id 2) (at 86.995 149.098 90)
@@
   (symbol (lib_id "Device:R") (at 108.585 56.515 0) (unit 1)
     (in_bom yes) (on_board yes)
-    (property "Reference" "R64" (id 0) (at 110.49 55.2449 0)
+    (property "Reference" "R20" (id 0) (at 110.49 55.2449 0)
       (effects (font (size 1.27 1.27)) (justify left))
     )
@@
   (symbol (lib_id "Device:R") (at 76.835 137.795 0) (unit 1)
     (in_bom yes) (on_board yes) (fields_autoplaced)
-    (property "Reference" "R77" (id 0) (at 79.375 136.5249 0)
+    (property "Reference" "R63" (id 0) (at 79.375 136.5249 0)
       (effects (font (size 1.27 1.27)) (justify left))
     )
@@
   (symbol (lib_id "Device:R") (at 86.995 117.475 90) (unit 1)
     (in_bom yes) (on_board yes) (fields_autoplaced)
-    (property "Reference" "R75" (id 0) (at 86.995 111.125 90))
+    (property "Reference" "R62" (id 0) (at 86.995 111.125 90))
     (property "Value" "100K" (id 1) (at 86.995 113.665 90))
     (property "Footprint" "Resistor_THT:R_Axial_DIN0207_L6.3mm_D2.5mm_P7.62mm_Horizontal" (id 2) (at 86.995 119.253 90)
@@
   (symbol (lib_id "Transistor_BJT:2N3904") (at 106.045 78.105 0) (unit 1)
     (in_bom yes) (on_board yes) (fields_autoplaced)
-    (property "Reference" "Q13" (id 0) (at 111.76 76.8349 0)
+    (property "Reference" "Q5" (id 0) (at 111.76 76.8349 0)
       (effects (font (size 1.27 1.27)) (justify left))
     )
@@
   (symbol (lib_id "Amplifier_Operational:TL074") (at 189.865 66.04 0) (mirror x) (unit 2)
     (in_bom yes) (on_board yes)
-    (property "Reference" "U2" (id 0) (at 189.865 57.15 0))
+    (property "Reference" "U3" (id 0) (at 189.865 57.15 0))
     (property "Value" "TL074" (id 1) (at 189.865 59.69 0))
     (property "Footprint" "Package_SO:SOIC-14_3.9x8.7mm_P1.27mm" (id 2) (at 188.595 68.58 0)
@@
   (symbol (lib_id "Device:R") (at 108.585 133.985 90) (unit 1)
     (in_bom yes) (on_board yes) (fields_autoplaced)
-    (property "Reference" "R76" (id 0) (at 108.585 127.635 90))
+    (property "Reference" "R58" (id 0) (at 108.585 127.635 90))
     (property "Value" "52K" (id 1) (at 108.585 130.175 90))
     (property "Footprint" "Resistor_THT:R_Axial_DIN0207_L6.3mm_D2.5mm_P7.62mm_Horizontal" (id 2) (at 108.585 135.763 90)
@@
   (symbol (lib_id "Connector:Conn_01x02_Male") (at 71.12 73.025 90) (mirror x) (unit 1)
     (in_bom yes) (on_board yes) (fields_autoplaced)
-    (property "Reference" "J11" (id 0) (at 74.93 72.3899 90)
+    (property "Reference" "J6" (id 0) (at 74.93 72.3899 90)
       (effects (font (size 1.27 1.27)) (justify right))
     )
@@
   (symbol (lib_id "Device:R") (at 163.83 63.5 90) (unit 1)
     (in_bom yes) (on_board yes) (fields_autoplaced)
-    (property "Reference" "R66" (id 0) (at 163.83 57.785 90))
+    (property "Reference" "R67" (id 0) (at 163.83 57.785 90))
     (property "Value" "1K" (id 1) (at 163.83 60.325 90))
     (property "Footprint" "Resistor_THT:R_Axial_DIN0207_L6.3mm_D2.5mm_P7.62mm_Horizontal" (id 2) (at 163.83 65.278 90)
@@
   (symbol (lib_id "Connector:Conn_01x02_Male") (at 71.12 112.395 90) (mirror x) (unit 1)
     (in_bom yes) (on_board yes) (fields_autoplaced)
-    (property "Reference" "J12" (id 0) (at 74.93 111.7599 90)
+    (property "Reference" "J18" (id 0) (at 74.93 111.7599 90)
       (effects (font (size 1.27 1.27)) (justify right))
     )
@@
   (symbol (lib_id "Device:R") (at 86.995 78.105 90) (unit 1)
     (in_bom yes) (on_board yes) (fields_autoplaced)
-    (property "Reference" "R70" (id 0) (at 86.995 71.755 90))
+    (property "Reference" "R3" (id 0) (at 86.995 71.755 90))
     (property "Value" "100K" (id 1) (at 86.995 74.295 90))
     (property "Footprint" "Resistor_THT:R_Axial_DIN0207_L6.3mm_D2.5mm_P7.62mm_Horizontal" (id 2) (at 86.995 79.883 90)
@@
   (symbol (lib_id "Device:R") (at 163.83 68.58 90) (unit 1)
     (in_bom yes) (on_board yes)
-    (property "Reference" "R68" (id 0) (at 163.83 73.66 90))
+    (property "Reference" "R65" (id 0) (at 163.83 73.66 90))
     (property "Value" "1K" (id 1) (at 163.83 71.12 90))
     (property "Footprint" "Resistor_THT:R_Axial_DIN0207_L6.3mm_D2.5mm_P7.62mm_Horizontal" (id 2) (at 163.83 70.358 90)
@@
   (symbol (lib_id "Device:R") (at 156.21 78.105 90) (unit 1)
     (in_bom yes) (on_board yes) (fields_autoplaced)
-    (property "Reference" "R71" (id 0) (at 156.21 71.755 90))
+    (property "Reference" "R36" (id 0) (at 156.21 71.755 90))
     (property "Value" "100K" (id 1) (at 156.21 74.295 90))
     (property "Footprint" "Resistor_THT:R_Axial_DIN0207_L6.3mm_D2.5mm_P7.62mm_Horizontal" (id 2) (at 156.21 79.883 90)
@@
   (symbol (lib_id "Device:R_Potentiometer") (at 76.835 147.32 0) (unit 1)
     (in_bom yes) (on_board yes) (fields_autoplaced)
-    (property "Reference" "RV18" (id 0) (at 74.295 146.0499 0)
+    (property "Reference" "RV11" (id 0) (at 74.295 146.0499 0)
       (effects (font (size 1.27 1.27)) (justify right))
     )
@@
   (symbol (lib_id "Device:R_Potentiometer_Trim") (at 168.275 97.155 90) (unit 1)
     (in_bom yes) (on_board yes) (fields_autoplaced)
-    (property "Reference" "RV17" (id 0) (at 168.275 100.33 90))
+    (property "Reference" "RV10" (id 0) (at 168.275 100.33 90))
     (property "Value" "100K" (id 1) (at 168.275 102.87 90))
     (property "Footprint" "SloBlo:Potentiometer_Bourns_3296W_Vertical" (id 2) (at 168.275 97.155 0)
@@
   (symbol (lib_id "Transistor_BJT:2N3904") (at 134.62 78.105 0) (mirror y) (unit 1)
     (in_bom yes) (on_board yes) (fields_autoplaced)
-    (property "Reference" "Q14" (id 0) (at 129.54 76.8349 0)
+    (property "Reference" "Q6" (id 0) (at 129.54 76.8349 0)
       (effects (font (size 1.27 1.27)) (justify left))
     )
@@
   (symbol (lib_id "Device:R") (at 189.23 50.8 270) (unit 1)
     (in_bom yes) (on_board yes) (fields_autoplaced)
-    (property "Reference" "R63" (id 0) (at 189.23 45.085 90))
+    (property "Reference" "R66" (id 0) (at 189.23 45.085 90))
     (property "Value" "100K" (id 1) (at 189.23 47.625 90))
     (property "Footprint" "Resistor_THT:R_Axial_DIN0207_L6.3mm_D2.5mm_P7.62mm_Horizontal" (id 2) (at 189.23 49.022 90)
@@
   (symbol (lib_id "Device:R") (at 177.8 74.93 180) (unit 1)
     (in_bom yes) (on_board yes) (fields_autoplaced)
-    (property "Reference" "R69" (id 0) (at 179.705 73.6599 0)
+    (property "Reference" "R60" (id 0) (at 179.705 73.6599 0)
       (effects (font (size 1.27 1.27)) (justify right))
     )
@@
   (symbol (lib_id "Device:R") (at 145.415 86.995 0) (unit 1)
     (in_bom yes) (on_board yes) (fields_autoplaced)
-    (property "Reference" "R72" (id 0) (at 147.955 85.7249 0)
+    (property "Reference" "R18" (id 0) (at 147.955 85.7249 0)
       (effects (font (size 1.27 1.27)) (justify left))
     )
@@
   (symbol (lib_id "Device:R") (at 76.835 157.48 0) (unit 1)
     (in_bom yes) (on_board yes) (fields_autoplaced)
-    (property "Reference" "R79" (id 0) (at 79.375 156.2099 0)
+    (property "Reference" "R57" (id 0) (at 79.375 156.2099 0)
       (effects (font (size 1.27 1.27)) (justify left))
     )
@@
   (symbol (lib_id "Amplifier_Operational:TL074") (at 109.855 149.86 0) (mirror x) (unit 1)
     (in_bom yes) (on_board yes)
-    (property "Reference" "U2" (id 0) (at 109.855 140.97 0))
+    (property "Reference" "U3" (id 0) (at 109.855 140.97 0))
     (property "Value" "TL074" (id 1) (at 109.855 143.51 0))
     (property "Footprint" "Package_SO:SOIC-14_3.9x8.7mm_P1.27mm" (id 2) (at 108.585 152.4 0)
@@
   (symbol (lib_id "Device:R") (at 208.28 66.04 90) (unit 1)
     (in_bom yes) (on_board yes) (fields_autoplaced)
-    (property "Reference" "R67" (id 0) (at 208.28 60.325 90))
+    (property "Reference" "R35" (id 0) (at 208.28 60.325 90))
     (property "Value" "1K" (id 1) (at 208.28 62.865 90))
     (property "Footprint" "Resistor_THT:R_Axial_DIN0207_L6.3mm_D2.5mm_P7.62mm_Horizontal" (id 2) (at 208.28 67.818 90)
