File: hardware/KiCad/LivSynth_0v1/VCF.kicad_sch (KiCad schematic)
At the start: 34 parts, among them J10 Jumper, Q11 2N3906, Q12 2N3906, U12 TL074, U13 TL074, U6 LM13700

Commit message: Initial Routing finished
Parts:
- added J20, J9: Jumper, Connector_PinHeader_2.54mm:PinHeader_1x02_P2.54mm_Vertical, symbol Connector:Conn_01x02_Male
- added R126: 100K, Resistor_THT:R_Axial_DIN0207_L6.3mm_D2.5mm_P7.62mm_Horizontal, symbol Device:R
- RV15, RV16: footprint (none) -> SloBlo:RV141F-40-20BL
- U5: renamed from U12; footprint (none) -> Package_SO:SOIC-14_3.9x8.7mm_P1.27mm
- U5: renamed from U13; footprint (none) -> Package_SO:SOIC-14_3.9x8.7mm_P1.27mm
- U6: footprint (none) -> Package_SO:SOP-16_3.9x9.9mm_P1.27mm
Connections:
- net VCF_IN: now also J9.1 (Pin_1); no longer R49.1
- net VGND: now also U5.12 (+); no longer U5.3 (+)
- net at Q11.2 (B), R47.2, R55.2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: now also R126.2
- net at C39.1, R46.2, R54.2: now also U6.8; no longer U6.9
- net at C38.1, Q11.3 (C), R59.2: now also U5.13 (-); no longer U5.2 (-)
- net at C38.2, R48.2: now also U5.14; no longer U5.1
- net at D7.1 (K), D8.2 (A), R60.2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: now also U5.9 (-); no longer U5.2 (-)
- net at C40.2, D7.2 (A), D8.1 (K)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: now also U5.8; no longer U5.1
- net at R49.2, R51.2: now also U6.14 (+); no longer U6.3 (+)
- net at R61.2, RV16.2: now also U5.10 (+); no longer U5.3 (+)
- net at R45.1, R46.1: now also U6.4 (-); no longer U6.13 (-)
- net at R50.2, R53.2: now also U6.3 (+); no longer U6.14 (+)
- net at R44.2, R50.1, R52.2: now also U6.9; no longer U6.8
- net at R43.1, R44.1: now also U6.13 (-); no longer U6.4 (-)
- net VCF_EXP_CV_IN renamed VCF_CV1_IN
- new net: R57.1, U6.1, U6.16
- new net: J9.2 (Pin_2), R49.1
- new net: C40.1, U6.10, U6.12
- new net: J20.2 (Pin_2), R126.1
- new net: C41.1, U6.5, U6.7
- new net VCF_CV2_IN: J20.1 (Pin_1)
Other:
- moved on the sheet: J10, R47

Commit message: Rework for polyester film capacitors
Parts:
- C40, C41: footprint Capacitor_THT:C_Disc_D3.0mm_W1.6mm_P2.50mm -> Capacitor_THT:C_Rect_L7.2mm_W2.5mm_P5.00mm_FKS2_FKP2_MKS2_MKP2
Changed lines of the file:
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@@
       (effects (font (size 1.27 1.27)) (justify left))
     )
-    (property "Footprint" "Capacitor_THT:C_Disc_D3.0mm_W1.6mm_P2.50mm" (id 2) (at 169.8752 73.66 0)
+    (property "Footprint" "Capacitor_THT:C_Rect_L7.2mm_W2.5mm_P5.00mm_FKS2_FKP2_MKS2_MKP2" (id 2) (at 169.8752 73.66 0)
       (effects (font (size 1.27 1.27)) hide)
     )
@@
       (effects (font (size 1.27 1.27)) (justify left))
     )
-    (property "Footprint" "Capacitor_THT:C_Disc_D3.0mm_W1.6mm_P2.50mm" (id 2) (at 220.6752 73.66 0)
+    (property "Footprint" "Capacitor_THT:C_Rect_L7.2mm_W2.5mm_P5.00mm_FKS2_FKP2_MKS2_MKP2" (id 2) (at 220.6752 73.66 0)
       (effects (font (size 1.27 1.27)) hide)
     )

Commit message: Use correct Elko sizes (8mm/3.5mm)
Parts:
- C39: footprint Capacitor_THT:CP_Radial_D8.0mm_P5.00mm -> Capacitor_THT:CP_Radial_D8.0mm_P3.50mm
Changed lines of the file:
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@@
     (property "Reference" "C39" (id 0) (at 245.491 55.88 90))
     (property "Value" "33u" (id 1) (at 245.491 58.42 90))
-    (property "Footprint" "Capacitor_THT:CP_Radial_D8.0mm_P5.00mm" (id 2) (at 250.19 62.5348 0)
+    (property "Footprint" "Capacitor_THT:CP_Radial_D8.0mm_P3.50mm" (id 2) (at 250.19 62.5348 0)
       (effects (font (size 1.27 1.27)) hide)
     )

Commit message: 0v1 Ready for Production
Parts:
- C27: renamed from C41; value ${VCF_C_Value} -> 1n
- C30: renamed from C40; value ${VCF_C_Value} -> 1n
- R71: renamed from R45; value ${VCF_Rsmall_Value} -> 200
- R74: renamed from R50; value ${VCF_Rbig_Value} -> 10K
- R76: renamed from R43; value ${VCF_Rsmall_Value} -> 200
- R77: renamed from R49; value ${VCF_Rbig_Value} -> 10K
- R87: renamed from R46; value ${VCF_Rbig_Value} -> 10K
- R88: renamed from R51; value ${VCF_Rsmall_Value} -> 200
- R89: renamed from R44; value ${VCF_Rbig_Value} -> 10K
- R90: renamed from R52; value ${VCF_Rbig_Value} -> 10K
- R91: renamed from R53; value ${VCF_Rsmall_Value} -> 200
- R92: renamed from R54; value ${VCF_Rbig_Value} -> 10K
- renumbered C39 to C11, C38 to C13, D8 to D10, D7 to D4, J9 to J14, J20 to J8, J10 to J9, Q11 to Q10, Q12 to Q9, R47 to R25, R55 to R26, R126 to R28, R56 to R29, R60 to R30, R57 to R44, R58 to R47, R59 to R49, R62 to R52, R61 to R75, RV15 to RV3, RV16 to RV7, U5 to U6, U6 to U7
