File: hardware/KiCad/LivSynth_0v1/VCO.kicad_sch (KiCad schematic)
At the start: 33 parts, among them J6 Jumper, J7 Jumper, J8 Jumper, J9 Jumper, Q10 2N3904, Q8 2N3904, Q9 2N3904, SW6 SW_SPDT, U10 TL074, U11 TL074, U3 TL074, U4 TL074, U5 TL074

Commit message: Initial Routing finished
Parts:
- removed C37: 100n, Capacitor_THT:C_Disc_D3.0mm_W1.6mm_P2.50mm, symbol Device:C
- removed J9: Jumper, Connector_PinHeader_2.54mm:PinHeader_1x02_P2.54mm_Vertical, symbol Connector:Conn_01x02_Male
- removed R41: 10K, Resistor_THT:R_Axial_DIN0207_L6.3mm_D2.5mm_P7.62mm_Horizontal, symbol Device:R
- removed R42: 1M, Resistor_THT:R_Axial_DIN0207_L6.3mm_D2.5mm_P7.62mm_Horizontal, symbol Device:R
- removed RV10: 100K, symbol Device:R_Potentiometer
- added RV10: 100, Potentiometer_THT:Potentiometer_Bourns_3296W_Vertical, symbol Device:R_Potentiometer_Trim
- RV11, RV13, RV14: footprint (none) -> Potentiometer_THT:Potentiometer_Bourns_3296W_Vertical
- RV12: value 100 -> 100K; footprint (none) -> Potentiometer_THT:Potentiometer_Bourns_3296W_Vertical
- SW6: footprint (none) -> SloBlo:SW_Toggle_MS500C
- TH1: footprint (none) -> Resistor_THT:R_Axial_DIN0207_L6.3mm_D2.5mm_P7.62mm_Horizontal
- U3: renamed from U11; footprint (none) -> Package_SO:SOIC-14_3.9x8.7mm_P1.27mm
- U4: renamed from U3; footprint (none) -> Package_SO:SOIC-14_3.9x8.7mm_P1.27mm
- U4: renamed from U10; footprint (none) -> Package_SO:SOIC-14_3.9x8.7mm_P1.27mm
- U4: renamed from U5; footprint (none) -> Package_SO:SOIC-14_3.9x8.7mm_P1.27mm
- U4: footprint (none) -> Package_SO:SOIC-14_3.9x8.7mm_P1.27mm
Connections:
- net +9V: now also RV10.1
- net GND: now also RV10.3
- net SAW_OUT: now also U3.9 (-), U4.7; no longer U4.1
- net VCO_OUT: now also SW6.2 (B)
- net VGND: now also U3.10 (+), U4.10 (+), U4.5 (+); no longer U4.3 (+), U4.3 (+)
- net at C36.2, R39.2: now also U4.8; no longer U4.1
- net at C36.1, Q9.3 (C), R34.2: now also U4.9 (-); no longer U4.2 (-)
- net at RV14.1: now also U3.8; no longer U3.1
- net at RV13.2: now also U4.13 (-); no longer U4.2 (-)
- net at R38.1: now also RV10.2
- net at C35.1, Q10.3 (C), Q8.1 (E): now also U4.6 (-); no longer U4.2 (-)
- net at C34.2, Q8.2 (B): now also U4.14; no longer U4.1
- net at C34.1, RV12.2, RV12.3: now also U4.12 (+); no longer U4.3 (+)
Other:
- note added: "Fine Tune"
- note added: "Tracking"
- moved on the sheet: SW6, U3C

Commit message: Rework for polyester film capacitors
Parts:
- C34, C35: footprint Capacitor_THT:C_Disc_D3.0mm_W1.6mm_P2.50mm -> Capacitor_THT:C_Rect_L7.2mm_W2.5mm_P5.00mm_FKS2_FKP2_MKS2_MKP2
- RV10, RV11, RV12, RV13, RV14: footprint Potentiometer_THT:Potentiometer_Bourns_3296W_Vertical -> SloBlo:Potentiometer_Bourns_3296W_Vertical
Changed lines of the file:
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@@
       (effects (font (size 1.27 1.27)) (justify right))
     )
-    (property "Footprint" "Potentiometer_THT:Potentiometer_Bourns_3296W_Vertical" (id 2) (at 198.755 109.22 0)
+    (property "Footprint" "SloBlo:Potentiometer_Bourns_3296W_Vertical" (id 2) (at 198.755 109.22 0)
       (effects (font (size 1.27 1.27)) hide)
     )
@@
       (effects (font (size 1.27 1.27)) (justify right))
     )
-    (property "Footprint" "Potentiometer_THT:Potentiometer_Bourns_3296W_Vertical" (id 2) (at 95.885 82.55 0)
+    (property "Footprint" "SloBlo:Potentiometer_Bourns_3296W_Vertical" (id 2) (at 95.885 82.55 0)
       (effects (font (size 1.27 1.27)) hide)
     )
@@
     (property "Reference" "C35" (id 0) (at 173.355 62.23 90))
     (property "Value" "100n" (id 1) (at 173.355 64.77 90))
-    (property "Footprint" "Capacitor_THT:C_Disc_D3.0mm_W1.6mm_P2.50mm" (id 2) (at 177.165 68.8848 0)
+    (property "Footprint" "Capacitor_THT:C_Rect_L7.2mm_W2.5mm_P5.00mm_FKS2_FKP2_MKS2_MKP2" (id 2) (at 177.165 68.8848 0)
       (effects (font (size 1.27 1.27)) hide)
     )
@@
     (property "Reference" "RV12" (id 0) (at 196.215 86.36 90))
     (property "Value" "100K" (id 1) (at 196.215 88.9 90))
-    (property "Footprint" "Potentiometer_THT:Potentiometer_Bourns_3296W_Vertical" (id 2) (at 196.215 82.55 0)
+    (property "Footprint" "SloBlo:Potentiometer_Bourns_3296W_Vertical" (id 2) (at 196.215 82.55 0)
       (effects (font (size 1.27 1.27)) hide)
     )
@@
     (property "Reference" "C34" (id 0) (at 216.535 60.96 90))
     (property "Value" "1n" (id 1) (at 216.535 63.5 90))
-    (property "Footprint" "Capacitor_THT:C_Disc_D3.0mm_W1.6mm_P2.50mm" (id 2) (at 220.345 67.6148 0)
+    (property "Footprint" "Capacitor_THT:C_Rect_L7.2mm_W2.5mm_P5.00mm_FKS2_FKP2_MKS2_MKP2" (id 2) (at 220.345 67.6148 0)
       (effects (font (size 1.27 1.27)) hide)
     )
@@
       (effects (font (size 1.27 1.27)) (justify right))
     )
-    (property "Footprint" "Potentiometer_THT:Potentiometer_Bourns_3296W_Vertical" (id 2) (at 45.085 80.01 0)
+    (property "Footprint" "SloBlo:Potentiometer_Bourns_3296W_Vertical" (id 2) (at 45.085 80.01 0)
       (effects (font (size 1.27 1.27)) hide)
     )
@@
       (effects (font (size 1.27 1.27)) (justify right))
     )
-    (property "Footprint" "Potentiometer_THT:Potentiometer_Bourns_3296W_Vertical" (id 2) (at 189.865 135.89 0)
-      (effects (font (size 1.27 1.27)) hide)
-    )
+    (property "Footprint" "SloBlo:Potentiometer_Bourns_3296W_Vertical" (id 2) (at 189.865 135.89 0)
+      (effects (font (size 1.27 1.27)) hide)
+    )

Commit message: 0v1 Ready for Production
Parts:
- renumbered C35 to C14, C36 to C16, C34 to C17, J6 to J12, J7 to J13, J8 to J15, Q10 to Q12, Q9 to Q13, Q8 to Q14, R38 to R31, R39 to R32, R35 to R50, R33 to R51, R34 to R53, R36 to R54, R37 to R55, R40 to R78, RV11 to RV13, RV13 to RV16, RV14 to RV17, RV10 to RV2, SW6 to SW1, U3 to U8
Changed lines of the file:
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@@
   (symbol (lib_id "Device:R") (at 73.025 62.865 90) (unit 1)
     (in_bom yes) (on_board yes) (fields_autoplaced)
-    (property "Reference" "R37" (id 0) (at 73.025 56.515 90))
+    (property "Reference" "R55" (id 0) (at 73.025 56.515 90))
     (property "Value" "100K" (id 1) (at 73.025 59.055 90))
     (property "Footprint" "Resistor_THT:R_Axial_DIN0207_L6.3mm_D2.5mm_P7.62mm_Horizontal" (id 2) (at 73.025 64.643 90)
@@
   (symbol (lib_id "Connector:Conn_01x02_Male") (at 55.245 46.355 90) (mirror x) (unit 1)
     (in_bom yes) (on_board yes) (fields_autoplaced)
-    (property "Reference" "J7" (id 0) (at 59.69 45.7199 90)
+    (property "Reference" "J13" (id 0) (at 59.69 45.7199 90)
       (effects (font (size 1.27 1.27)) (justify right))
     )
@@
   (symbol (lib_id "Device:R") (at 182.245 62.23 0) (unit 1)
     (in_bom yes) (on_board yes) (fields_autoplaced)
-    (property "Reference" "R36" (id 0) (at 184.785 60.9599 0)
+    (property "Reference" "R54" (id 0) (at 184.785 60.9599 0)
       (effects (font (size 1.27 1.27)) (justify left))
     )
@@
   (symbol (lib_id "Device:R") (at 131.445 85.09 0) (unit 1)
     (in_bom yes) (on_board yes) (fields_autoplaced)
-    (property "Reference" "R39" (id 0) (at 133.985 83.8199 0)
+    (property "Reference" "R32" (id 0) (at 133.985 83.8199 0)
       (effects (font (size 1.27 1.27)) (justify left))
     )
@@
   (symbol (lib_id "Device:C") (at 121.285 93.98 90) (unit 1)
     (in_bom yes) (on_board yes) (fields_autoplaced)
-    (property "Reference" "C36" (id 0) (at 121.285 86.36 90))
+    (property "Reference" "C16" (id 0) (at 121.285 86.36 90))
     (property "Value" "1p" (id 1) (at 121.285 88.9 90))
     (property "Footprint" "Capacitor_THT:C_Disc_D3.0mm_W1.6mm_P2.50mm" (id 2) (at 125.095 93.0148 0)
@@
   (symbol (lib_id "Amplifier_Operational:TL074") (at 175.26 129.54 0) (unit 3)
     (in_bom yes) (on_board yes)
-    (property "Reference" "U3" (id 0) (at 175.26 138.43 0))
+    (property "Reference" "U8" (id 0) (at 175.26 138.43 0))
     (property "Value" "TL074" (id 1) (at 175.26 135.89 0))
     (property "Footprint" "Package_SO:SOIC-14_3.9x8.7mm_P1.27mm" (id 2) (at 173.99 127 0)
@@
   (symbol (lib_id "Device:R") (at 73.025 51.435 90) (unit 1)
     (in_bom yes) (on_board yes) (fields_autoplaced)
-    (property "Reference" "R35" (id 0) (at 73.025 45.085 90))
+    (property "Reference" "R50" (id 0) (at 73.025 45.085 90))
     (property "Value" "100K" (id 1) (at 73.025 47.625 90))
     (property "Footprint" "Resistor_THT:R_Axial_DIN0207_L6.3mm_D2.5mm_P7.62mm_Horizontal" (id 2) (at 73.025 53.213 90)
@@
   (symbol (lib_id "Device:R_Potentiometer_Trim") (at 198.755 109.22 0) (unit 1)
     (in_bom yes) (on_board yes) (fields_autoplaced)
-    (property "Reference" "RV13" (id 0) (at 196.215 107.9499 0)
+    (property "Reference" "RV16" (id 0) (at 196.215 107.9499 0)
       (effects (font (size 1.27 1.27)) (justify right))
     )
@@
   (symbol (lib_id "Transistor_BJT:2N3904") (at 145.415 69.85 0) (mirror y) (unit 1)
     (in_bom yes) (on_board yes) (fields_autoplaced)
-    (property "Reference" "Q10" (id 0) (at 140.335 68.5799 0)
+    (property "Reference" "Q12" (id 0) (at 140.335 68.5799 0)
       (effects (font (size 1.27 1.27)) (justify left))
     )
@@
   (symbol (lib_id "Device:R_Potentiometer_Trim") (at 95.885 82.55 0) (unit 1)
     (in_bom yes) (on_board yes) (fields_autoplaced)
-    (property "Reference" "RV11" (id 0) (at 93.345 81.2799 0)
+    (property "Reference" "RV13" (id 0) (at 93.345 81.2799 0)
       (effects (font (size 1.27 1.27)) (justify right))
     )
@@
   (symbol (lib_id "Device:R") (at 73.025 73.66 90) (unit 1)
     (in_bom yes) (on_board yes) (fields_autoplaced)
-    (property "Reference" "R38" (id 0) (at 73.025 67.31 90))
+    (property "Reference" "R31" (id 0) (at 73.025 67.31 90))
     (property "Value" "100K" (id 1) (at 73.025 69.85 90))
     (property "Footprint" "Resistor_THT:R_Axial_DIN0207_L6.3mm_D2.5mm_P7.62mm_Horizontal" (id 2) (at 73.025 75.438 90)
@@
   (symbol (lib_id "Device:C") (at 173.355 69.85 90) (unit 1)
     (in_bom yes) (on_board yes) (fields_autoplaced)
-    (property "Reference" "C35" (id 0) (at 173.355 62.23 90))
+    (property "Reference" "C14" (id 0) (at 173.355 62.23 90))
     (property "Value" "100n" (id 1) (at 173.355 64.77 90))
     (property "Footprint" "Capacitor_THT:C_Rect_L7.2mm_W2.5mm_P5.00mm_FKS2_FKP2_MKS2_MKP2" (id 2) (at 177.165 68.8848 0)
@@
   (symbol (lib_id "Transistor_BJT:2N3904") (at 173.355 50.8 270) (unit 1)
     (in_bom yes) (on_board yes) (fields_autoplaced)
-    (property "Reference" "Q8" (id 0) (at 173.355 57.15 90))
+    (property "Reference" "Q14" (id 0) (at 173.355 57.15 90))
     (property "Value" "2N3904" (id 1) (at 173.355 59.69 90))
     (property "Footprint" "Package_TO_SOT_THT:TO-92_Inline" (id 2) (at 171.45 55.88 0)
@@
   (symbol (lib_id "Connector:Conn_01x02_Male") (at 55.245 57.785 90) (mirror x) (unit 1)
     (in_bom yes) (on_board yes) (fields_autoplaced)
-    (property "Reference" "J8" (id 0) (at 59.69 57.1499 90)
+    (property "Reference" "J15" (id 0) (at 59.69 57.1499 90)
       (effects (font (size 1.27 1.27)) (justify right))
     )
@@
   (symbol (lib_id "Device:C") (at 216.535 68.58 90) (unit 1)
     (in_bom yes) (on_board yes) (fields_autoplaced)
-    (property "Reference" "C34" (id 0) (at 216.535 60.96 90))
+    (property "Reference" "C17" (id 0) (at 216.535 60.96 90))
     (property "Value" "1n" (id 1) (at 216.535 63.5 90))
     (property "Footprint" "Capacitor_THT:C_Rect_L7.2mm_W2.5mm_P5.00mm_FKS2_FKP2_MKS2_MKP2" (id 2) (at 220.345 67.6148 0)
@@
   (symbol (lib_id "Connector:Conn_01x02_Male") (at 55.245 34.925 90) (mirror x) (unit 1)
     (in_bom yes) (on_board yes) (fields_autoplaced)
-    (property "Reference" "J6" (id 0) (at 59.69 34.2899 90)
+    (property "Reference" "J12" (id 0) (at 59.69 34.2899 90)
       (effects (font (size 1.27 1.27)) (justify right))
     )
@@
   (symbol (lib_id "Switch:SW_SPDT") (at 241.3 125.73 0) (mirror y) (unit 1)
     (in_bom yes) (on_board yes) (fields_autoplaced)
-    (property "Reference" "SW6" (id 0) (at 241.3 118.11 0))
+    (property "Reference" "SW1" (id 0) (at 241.3 118.11 0))
     (property "Value" "SW_SPDT" (id 1) (at 241.3 120.65 0))
     (property "Footprint" "SloBlo:SW_Toggle_MS500C" (id 2) (at 241.3 125.73 0)
@@
   (symbol (lib_id "Device:R") (at 73.025 40.005 90) (unit 1)
     (in_bom yes) (on_board yes) (fields_autoplaced)
-    (property "Reference" "R33" (id 0) (at 73.025 33.655 90))
+    (property "Reference" "R51" (id 0) (at 73.025 33.655 90))
     (property "Value" "100K" (id 1) (at 73.025 36.195 90))
     (property "Footprint" "Resistor_THT:R_Axial_DIN0207_L6.3mm_D2.5mm_P7.62mm_Horizontal" (id 2) (at 73.025 41.783 90)
@@
   (symbol (lib_id "Device:R_Potentiometer_Trim") (at 45.085 80.01 0) (unit 1)
     (in_bom yes) (on_board yes) (fields_autoplaced)
-    (property "Reference" "RV10" (id 0) (at 42.545 78.7399 0)
+    (property "Reference" "RV2" (id 0) (at 42.545 78.7399 0)
       (effects (font (size 1.27 1.27)) (justify right))
     )
@@
   (symbol (lib_id "Transistor_BJT:2N3904") (at 117.475 69.85 0) (unit 1)
     (in_bom yes) (on_board yes) (fields_autoplaced)
-    (property "Reference" "Q9" (id 0) (at 122.555 68.5799 0)
+    (property "Reference" "Q13" (id 0) (at 122.555 68.5799 0)
       (effects (font (size 1.27 1.27)) (justify left))
     )
@@
   (symbol (lib_id "Device:R") (at 95.885 93.98 0) (unit 1)
     (in_bom yes) (on_board yes) (fields_autoplaced)
-    (property "Reference" "R40" (id 0) (at 98.425 92.7099 0)
+    (property "Reference" "R78" (id 0) (at 98.425 92.7099 0)
       (effects (font (size 1.27 1.27)) (justify left))
     )
@@
   (symbol (lib_id "Device:R") (at 109.855 44.45 0) (unit 1)
     (in_bom yes) (on_board yes)
-    (property "Reference" "R34" (id 0) (at 112.395 43.1799 0)
+    (property "Reference" "R53" (id 0) (at 112.395 43.1799 0)
       (effects (font (size 1.27 1.27)) (justify left))
     )
@@
   (symbol (lib_id "Device:R_Potentiometer_Trim") (at 189.865 135.89 0) (unit 1)
     (in_bom yes) (on_board yes) (fields_autoplaced)
-    (property "Reference" "RV14" (id 0) (at 187.325 134.6199 0)
-      (effects (font (size 1.27 1.27)) (justify right))
-    )
+    (property "Reference" "RV17" (id 0) (at 187.325 134.6199 0)
+      (effects (font (size 1.27 1.27)) (justify right))
+    )
