File: hardware/KiCad/LivSynth_0v2/LivSynth_Faceplate.kicad_pcb (KiCad board)
At the start: 2 copper layers, 230 x 159.9 mm, 85 parts, among them J1 PJ398SM, J2 PJ398SM, J3 PJ398SM, J7 Barrel_Jack_Switch, SW1 SW_SPDT, SW2 SW_SPST, SW3 SW_SPDT, SW4 SW_SPDT, SW6 SW_Push, SW7 SW_SPDT

Commit message: Speaker grill ready Test knob spin silkscreen with KiCad tools
Parts:
- removed J1, J2, J3: PJ398SM, SloBlo:Thonkiconn_PJ398SM
- removed LS1: LSM-50M/NO-B 8R (<32R) 1W, SloBlo:LSM-50M NO-B
- removed RGB_Pot1, RGB_Pot2, RGB_Pot3, RGB_Pot4, RGB_Pot5, RGB_Pot6, RGB_Pot7, RGB_Pot8, RGB_Pot9: TC002-N11AS2XT-RGB, SloBlo:TC002-N11AS2XT-RGB
- removed RV1: 1K, SloBlo:Potentiometer_Bourns_3296W_Vertical
- removed RV10, RV5, RV6, RV7: 100K, SloBlo:RV141F-40-20BL
- removed RV11: 100k, SloBlo:RV141F-40-20BL
- removed RV12, RV2: 100, SloBlo:Potentiometer_Bourns_3296W_Vertical
- removed RV13, RV14, RV18, RV19, RV20, RV22, RV3, RV8: 100K, SloBlo:Alpha_RD901F
- removed RV15, RV16, RV17: 100K, SloBlo:Potentiometer_Bourns_3296W_Vertical
- removed RV21: 10K, SloBlo:Alpha_RD901F
- removed RV4, RV9: 10K, SloBlo:RV141F-40-20BL
- removed SW1, SW3, SW4: SW_SPDT, SloBlo:SW_Toggle_MS500C
- removed SW2: SW_SPST, SloBlo:SW_Toggle_MS500C
- removed SW6: SW_Push, SloBlo:E-Switch_TL1105SP
- added REF**: Via 1mm, SloBloFP:Via 1mm, F.Cu at (242.5, 85.9)
- added REF**: Via 1mm, SloBloFP:Via 1mm, F.Cu at (240.5, 87.9)
- added REF**: Via 1mm, SloBloFP:Via 1mm, F.Cu at (237.5, 87.9)
- added REF**1: Via 1mm, SloBloFP:Via 1mm, F.Cu at (239.6, 85.8)
- added REF**10: Via 1mm, SloBloFP:Via 1mm, F.Cu at (235.5, 82.9)
- added REF**100: Via 1mm, SloBloFP:Via 1mm, F.Cu at (224.6, 95.6)
- added REF**101: Via 1mm, SloBloFP:Via 1mm, F.Cu at (226.2, 97.9)
- added REF**102: Via 1mm, SloBloFP:Via 1mm, F.Cu at (228.3, 99.8)
- added REF**103: Via 1mm, SloBloFP:Via 1mm, F.Cu at (230.6, 101.3)
- added REF**104: Via 1mm, SloBloFP:Via 1mm, F.Cu at (233.2, 102.3)
- added REF**105: Via 1mm, SloBloFP:Via 1mm, F.Cu at (235.9, 102.9)
- added REF**106: Via 1mm, SloBloFP:Via 1mm, F.Cu at (238.7, 102.9)
- added REF**107: Via 1mm, SloBloFP:Via 1mm, F.Cu at (241.4, 102.4)
- added REF**108: Via 1mm, SloBloFP:Via 1mm, F.Cu at (244.0, 101.5)
- added REF**109: Via 1mm, SloBloFP:Via 1mm, F.Cu at (246.4, 100.1)
- added REF**11: Via 1mm, SloBloFP:Via 1mm, F.Cu at (233.3, 84.6)
- added REF**110: Via 1mm, SloBloFP:Via 1mm, F.Cu at (248.5, 98.2)
- added REF**111: Via 1mm, SloBloFP:Via 1mm, F.Cu at (250.2, 96.0)
- added REF**112: Via 1mm, SloBloFP:Via 1mm, F.Cu at (251.5, 93.6)
- added REF**113: Via 1mm, SloBloFP:Via 1mm, F.Cu at (252.3, 90.9)
- added REF**114: Via 1mm, SloBloFP:Via 1mm, F.Cu at (252.6, 88.1)
- added REF**115: Via 1mm, SloBloFP:Via 1mm, F.Cu at (254.7, 83.7)
- added REF**116: Via 1mm, SloBloFP:Via 1mm, F.Cu at (253.8, 81.0)
- added REF**117: Via 1mm, SloBloFP:Via 1mm, F.Cu at (252.6, 78.6)
- added REF**118: Via 1mm, SloBloFP:Via 1mm, F.Cu at (250.9, 76.3)
- added REF**119: Via 1mm, SloBloFP:Via 1mm, F.Cu at (248.9, 74.4)
- added REF**12: Via 1mm, SloBloFP:Via 1mm, F.Cu at (232.2, 87.2)
- added REF**120: Via 1mm, SloBloFP:Via 1mm, F.Cu at (246.7, 72.7)
- added REF**121: Via 1mm, SloBloFP:Via 1mm, F.Cu at (244.2, 71.5)
- added REF**122: Via 1mm, SloBloFP:Via 1mm, F.Cu at (241.5, 70.7)
- added REF**123: Via 1mm, SloBloFP:Via 1mm, F.Cu at (238.8, 70.2)
- added REF**124: Via 1mm, SloBloFP:Via 1mm, F.Cu at (236.0, 70.3)
- added REF**125: Via 1mm, SloBloFP:Via 1mm, F.Cu at (233.3, 70.7)
- added REF**126: Via 1mm, SloBloFP:Via 1mm, F.Cu at (230.6, 71.6)
- added REF**127: Via 1mm, SloBloFP:Via 1mm, F.Cu at (228.2, 72.9)
- added REF**128: Via 1mm, SloBloFP:Via 1mm, F.Cu at (225.9, 74.5)
- added REF**129: Via 1mm, SloBloFP:Via 1mm, F.Cu at (224.0, 76.5)
- added REF**13: Via 1mm, SloBloFP:Via 1mm, F.Cu at (232.5, 89.9)
- added REF**130: Via 1mm, SloBloFP:Via 1mm, F.Cu at (222.3, 78.8)
- added REF**131: Via 1mm, SloBloFP:Via 1mm, F.Cu at (221.1, 81.2)
- added REF**132: Via 1mm, SloBloFP:Via 1mm, F.Cu at (220.3, 83.9)
- added REF**133: Via 1mm, SloBloFP:Via 1mm, F.Cu at (219.8, 86.6)
- added REF**134: Via 1mm, SloBloFP:Via 1mm, F.Cu at (219.9, 89.4)
- added REF**135: Via 1mm, SloBloFP:Via 1mm, F.Cu at (220.3, 92.2)
- added REF**136: Via 1mm, SloBloFP:Via 1mm, F.Cu at (221.2, 94.8)
- added REF**137: Via 1mm, SloBloFP:Via 1mm, F.Cu at (222.5, 97.3)
- added REF**138: Via 1mm, SloBloFP:Via 1mm, F.Cu at (224.1, 99.5)
- added REF**139: Via 1mm, SloBloFP:Via 1mm, F.Cu at (226.1, 101.5)
- added REF**14: Via 1mm, SloBloFP:Via 1mm, F.Cu at (234.2, 92.2)
- added REF**140: Via 1mm, SloBloFP:Via 1mm, F.Cu at (228.3, 103.1)
- added REF**141: Via 1mm, SloBloFP:Via 1mm, F.Cu at (230.8, 104.3)
- added REF**142: Via 1mm, SloBloFP:Via 1mm, F.Cu at (233.5, 105.2)
- added REF**143: Via 1mm, SloBloFP:Via 1mm, F.Cu at (236.2, 105.6)
- added REF**144: Via 1mm, SloBloFP:Via 1mm, F.Cu at (239.0, 105.6)
- added REF**145: Via 1mm, SloBloFP:Via 1mm, F.Cu at (241.8, 105.1)
- added REF**146: Via 1mm, SloBloFP:Via 1mm, F.Cu at (244.4, 104.3)
- added REF**147: Via 1mm, SloBloFP:Via 1mm, F.Cu at (246.9, 103.0)
- added REF**148: Via 1mm, SloBloFP:Via 1mm, F.Cu at (249.1, 101.3)
- added REF**149: Via 1mm, SloBloFP:Via 1mm, F.Cu at (251.1, 99.3)
- added REF**15: Via 1mm, SloBloFP:Via 1mm, F.Cu at (236.7, 93.2)
- added REF**150: Via 1mm, SloBloFP:Via 1mm, F.Cu at (252.7, 97.1)
- added REF**151: Via 1mm, SloBloFP:Via 1mm, F.Cu at (253.9, 94.6)
- added REF**152: Via 1mm, SloBloFP:Via 1mm, F.Cu at (254.8, 91.9)
- added REF**153: Via 1mm, SloBloFP:Via 1mm, F.Cu at (255.2, 89.2)
- added REF**154: Via 1mm, SloBloFP:Via 1mm, F.Cu at (257.0, 82.1)
- added REF**155: Via 1mm, SloBloFP:Via 1mm, F.Cu at (256.1, 79.6)
- added REF**156: Via 1mm, SloBloFP:Via 1mm, F.Cu at (254.8, 77.3)
- added REF**157: Via 1mm, SloBloFP:Via 1mm, F.Cu at (253.3, 75.1)
- added REF**158: Via 1mm, SloBloFP:Via 1mm, F.Cu at (251.5, 73.2)
- added REF**159: Via 1mm, SloBloFP:Via 1mm, F.Cu at (249.4, 71.5)
- added REF**16: Via 1mm, SloBloFP:Via 1mm, F.Cu at (239.5, 92.9)
- added REF**160: Via 1mm, SloBloFP:Via 1mm, F.Cu at (247.2, 70.0)
- added REF**161: Via 1mm, SloBloFP:Via 1mm, F.Cu at (244.8, 68.9)
- added REF**162: Via 1mm, SloBloFP:Via 1mm, F.Cu at (242.2, 68.2)
- added REF**163: Via 1mm, SloBloFP:Via 1mm, F.Cu at (239.6, 67.7)
- added REF**164: Via 1mm, SloBloFP:Via 1mm, F.Cu at (236.9, 67.6)
- added REF**165: Via 1mm, SloBloFP:Via 1mm, F.Cu at (234.3, 67.9)
- added REF**166: Via 1mm, SloBloFP:Via 1mm, F.Cu at (231.7, 68.5)
- added REF**167: Via 1mm, SloBloFP:Via 1mm, F.Cu at (229.2, 69.4)
- added REF**168: Via 1mm, SloBloFP:Via 1mm, F.Cu at (226.9, 70.6)
- added REF**169: Via 1mm, SloBloFP:Via 1mm, F.Cu at (224.7, 72.2)
- added REF**17: Via 1mm, SloBloFP:Via 1mm, F.Cu at (241.7, 91.2)
- added REF**170: Via 1mm, SloBloFP:Via 1mm, F.Cu at (222.7, 74.0)
- added REF**171: Via 1mm, SloBloFP:Via 1mm, F.Cu at (221.1, 76.0)
- added REF**172: Via 1mm, SloBloFP:Via 1mm, F.Cu at (219.6, 78.3)
- added REF**173: Via 1mm, SloBloFP:Via 1mm, F.Cu at (218.5, 80.7)
- added REF**174: Via 1mm, SloBloFP:Via 1mm, F.Cu at (217.7, 83.2)
- added REF**175: Via 1mm, SloBloFP:Via 1mm, F.Cu at (217.3, 85.8)
- added REF**176: Via 1mm, SloBloFP:Via 1mm, F.Cu at (217.2, 88.5)
- added REF**177: Via 1mm, SloBloFP:Via 1mm, F.Cu at (217.5, 91.1)
- added REF**178: Via 1mm, SloBloFP:Via 1mm, F.Cu at (218.0, 93.7)
- added REF**179: Via 1mm, SloBloFP:Via 1mm, F.Cu at (219.0, 96.2)
- added REF**18: Via 1mm, SloBloFP:Via 1mm, F.Cu at (245.1, 86.9)
- added REF**18: Via 1mm, SloBloFP:Via 1mm, F.Cu at (242.8, 88.7)
- added REF**180: Via 1mm, SloBloFP:Via 1mm, F.Cu at (220.2, 98.6)
- added REF**181: Via 1mm, SloBloFP:Via 1mm, F.Cu at (221.8, 100.7)
- added REF**182: Via 1mm, SloBloFP:Via 1mm, F.Cu at (223.6, 102.7)
- added REF**183: Via 1mm, SloBloFP:Via 1mm, F.Cu at (225.6, 104.4)
- added REF**184: Via 1mm, SloBloFP:Via 1mm, F.Cu at (227.9, 105.8)
- added REF**185: Via 1mm, SloBloFP:Via 1mm, F.Cu at (230.3, 106.9)
- added REF**186: Via 1mm, SloBloFP:Via 1mm, F.Cu at (232.8, 107.7)
- added REF**187: Via 1mm, SloBloFP:Via 1mm, F.Cu at (235.4, 108.1)
- added REF**188: Via 1mm, SloBloFP:Via 1mm, F.Cu at (238.1, 108.2)
- added REF**189: Via 1mm, SloBloFP:Via 1mm, F.Cu at (240.7, 108.0)
- added REF**19: Via 1mm, SloBloFP:Via 1mm, F.Cu at (244.2, 84.1)
- added REF**190: Via 1mm, SloBloFP:Via 1mm, F.Cu at (243.3, 107.4)
- added REF**191: Via 1mm, SloBloFP:Via 1mm, F.Cu at (245.8, 106.5)
- added REF**192: Via 1mm, SloBloFP:Via 1mm, F.Cu at (248.2, 105.2)
- added REF**193: Via 1mm, SloBloFP:Via 1mm, F.Cu at (250.3, 103.7)
- added REF**194: Via 1mm, SloBloFP:Via 1mm, F.Cu at (252.3, 101.9)
- added REF**195: Via 1mm, SloBloFP:Via 1mm, F.Cu at (254.0, 99.8)
- added REF**196: Via 1mm, SloBloFP:Via 1mm, F.Cu at (255.4, 97.6)
- added REF**197: Via 1mm, SloBloFP:Via 1mm, F.Cu at (256.5, 95.2)
- added REF**198: Via 1mm, SloBloFP:Via 1mm, F.Cu at (257.3, 92.6)
- added REF**199: Via 1mm, SloBloFP:Via 1mm, F.Cu at (257.7, 90.0)
- added REF**2: Via 1mm, SloBloFP:Via 1mm, F.Cu at (237.5, 84.9)
- added REF**20: Via 1mm, SloBloFP:Via 1mm, F.Cu at (242.2, 81.8)
- added REF**200: Via 1mm, SloBloFP:Via 1mm, F.Cu at (260.4, 85.7)
- added REF**200: Via 1mm, SloBloFP:Via 1mm, F.Cu at (257.8, 87.3)
- added REF**201: Via 1mm, SloBloFP:Via 1mm, F.Cu at (260.1, 83.2)
- added REF**202: Via 1mm, SloBloFP:Via 1mm, F.Cu at (259.4, 80.7)
- added REF**203: Via 1mm, SloBloFP:Via 1mm, F.Cu at (258.4, 78.3)
- added REF**204: Via 1mm, SloBloFP:Via 1mm, F.Cu at (257.2, 76.0)
- added REF**205: Via 1mm, SloBloFP:Via 1mm, F.Cu at (255.8, 73.9)
- added REF**206: Via 1mm, SloBloFP:Via 1mm, F.Cu at (254.1, 71.9)
- added REF**207: Via 1mm, SloBloFP:Via 1mm, F.Cu at (252.2, 70.2)
- added REF**208: Via 1mm, SloBloFP:Via 1mm, F.Cu at (250.1, 68.6)
- added REF**209: Via 1mm, SloBloFP:Via 1mm, F.Cu at (247.9, 67.3)
- added REF**21: Via 1mm, SloBloFP:Via 1mm, F.Cu at (239.5, 80.5)
- added REF**210: Via 1mm, SloBloFP:Via 1mm, F.Cu at (245.5, 66.3)
- added REF**211: Via 1mm, SloBloFP:Via 1mm, F.Cu at (243.0, 65.6)
- added REF**212: Via 1mm, SloBloFP:Via 1mm, F.Cu at (240.5, 65.1)
- added REF**213: Via 1mm, SloBloFP:Via 1mm, F.Cu at (237.9, 64.9)
- added REF**214: Via 1mm, SloBloFP:Via 1mm, F.Cu at (235.3, 65.0)
- added REF**215: Via 1mm, SloBloFP:Via 1mm, F.Cu at (232.8, 65.4)
- added REF**216: Via 1mm, SloBloFP:Via 1mm, F.Cu at (230.3, 66.1)
- added REF**217: Via 1mm, SloBloFP:Via 1mm, F.Cu at (227.9, 67.0)
- added REF**218: Via 1mm, SloBloFP:Via 1mm, F.Cu at (225.6, 68.2)
- added REF**219: Via 1mm, SloBloFP:Via 1mm, F.Cu at (223.5, 69.7)
- added REF**22: Via 1mm, SloBloFP:Via 1mm, F.Cu at (236.5, 80.3)
- added REF**220: Via 1mm, SloBloFP:Via 1mm, F.Cu at (221.5, 71.4)
- added REF**221: Via 1mm, SloBloFP:Via 1mm, F.Cu at (219.8, 73.3)
- added REF**222: Via 1mm, SloBloFP:Via 1mm, F.Cu at (218.2, 75.3)
- added REF**223: Via 1mm, SloBloFP:Via 1mm, F.Cu at (216.9, 77.6)
- added REF**224: Via 1mm, SloBloFP:Via 1mm, F.Cu at (215.9, 79.9)
- added REF**225: Via 1mm, SloBloFP:Via 1mm, F.Cu at (215.2, 82.4)
- added REF**226: Via 1mm, SloBloFP:Via 1mm, F.Cu at (214.7, 85.0)
- added REF**227: Via 1mm, SloBloFP:Via 1mm, F.Cu at (214.5, 87.5)
- added REF**228: Via 1mm, SloBloFP:Via 1mm, F.Cu at (214.6, 90.1)
- added REF**229: Via 1mm, SloBloFP:Via 1mm, F.Cu at (215.0, 92.7)
- added REF**23: Via 1mm, SloBloFP:Via 1mm, F.Cu at (233.7, 81.2)
- added REF**230: Via 1mm, SloBloFP:Via 1mm, F.Cu at (215.7, 95.2)
- added REF**231: Via 1mm, SloBloFP:Via 1mm, F.Cu at (216.6, 97.6)
- added REF**232: Via 1mm, SloBloFP:Via 1mm, F.Cu at (217.8, 99.8)
- added REF**233: Via 1mm, SloBloFP:Via 1mm, F.Cu at (219.3, 102.0)
- added REF**234: Via 1mm, SloBloFP:Via 1mm, F.Cu at (221.0, 103.9)
- added REF**235: Via 1mm, SloBloFP:Via 1mm, F.Cu at (222.9, 105.7)
- added REF**236: Via 1mm, SloBloFP:Via 1mm, F.Cu at (224.9, 107.2)
- added REF**237: Via 1mm, SloBloFP:Via 1mm, F.Cu at (227.2, 108.5)
- added REF**238: Via 1mm, SloBloFP:Via 1mm, F.Cu at (229.5, 109.5)
- added REF**239: Via 1mm, SloBloFP:Via 1mm, F.Cu at (232.0, 110.3)
- added REF**24: Via 1mm, SloBloFP:Via 1mm, F.Cu at (231.4, 83.2)
- added REF**240: Via 1mm, SloBloFP:Via 1mm, F.Cu at (234.6, 110.8)
- added REF**241: Via 1mm, SloBloFP:Via 1mm, F.Cu at (237.1, 110.9)
- added REF**242: Via 1mm, SloBloFP:Via 1mm, F.Cu at (239.7, 110.8)
- added REF**243: Via 1mm, SloBloFP:Via 1mm, F.Cu at (242.3, 110.5)
- added REF**244: Via 1mm, SloBloFP:Via 1mm, F.Cu at (244.8, 109.8)
- added REF**245: Via 1mm, SloBloFP:Via 1mm, F.Cu at (247.2, 108.8)
- added REF**246: Via 1mm, SloBloFP:Via 1mm, F.Cu at (249.4, 107.6)
- added REF**247: Via 1mm, SloBloFP:Via 1mm, F.Cu at (251.6, 106.2)
- added REF**248: Via 1mm, SloBloFP:Via 1mm, F.Cu at (253.5, 104.5)
- added REF**249: Via 1mm, SloBloFP:Via 1mm, F.Cu at (255.3, 102.6)
- added REF**25: Via 1mm, SloBloFP:Via 1mm, F.Cu at (230.1, 85.9)
- added REF**250: Via 1mm, SloBloFP:Via 1mm, F.Cu at (256.8, 100.5)
- added REF**251: Via 1mm, SloBloFP:Via 1mm, F.Cu at (258.1, 98.2)
- added REF**252: Via 1mm, SloBloFP:Via 1mm, F.Cu at (259.1, 95.9)
- added REF**253: Via 1mm, SloBloFP:Via 1mm, F.Cu at (259.9, 93.4)
- added REF**254: Via 1mm, SloBloFP:Via 1mm, F.Cu at (260.4, 90.9)
- added REF**255: Via 1mm, SloBloFP:Via 1mm, F.Cu at (260.5, 88.3)
- added REF**26: Via 1mm, SloBloFP:Via 1mm, F.Cu at (229.9, 88.9)
- added REF**27: Via 1mm, SloBloFP:Via 1mm, F.Cu at (230.8, 91.7)
- added REF**28: Via 1mm, SloBloFP:Via 1mm, F.Cu at (232.8, 94.0)
- added REF**29: Via 1mm, SloBloFP:Via 1mm, F.Cu at (235.5, 95.3)
- added REF**3: Via 1mm, SloBloFP:Via 1mm, F.Cu at (235.4, 85.8)
- added REF**30: Via 1mm, SloBloFP:Via 1mm, F.Cu at (238.5, 95.6)
- added REF**31: Via 1mm, SloBloFP:Via 1mm, F.Cu at (241.3, 94.6)
- added REF**32: Via 1mm, SloBloFP:Via 1mm, F.Cu at (243.6, 92.6)
- added REF**33: Via 1mm, SloBloFP:Via 1mm, F.Cu at (249.9, 87.2)
- added REF**33: Via 1mm, SloBloFP:Via 1mm, F.Cu at (252.3, 85.4)
- added REF**33: Via 1mm, SloBloFP:Via 1mm, F.Cu at (244.9, 89.9)
- added REF**33: Via 1mm, SloBloFP:Via 1mm, F.Cu at (247.5, 88.7)
- added REF**33: Via 1mm, SloBloFP:Via 1mm, F.Cu at (257.6, 84.7)
- added REF**33: Via 1mm, SloBloFP:Via 1mm, F.Cu at (255.2, 86.4)
- added REF**34: Via 1mm, SloBloFP:Via 1mm, F.Cu at (247.3, 85.8)
- added REF**35: Via 1mm, SloBloFP:Via 1mm, F.Cu at (246.3, 83.1)
- added REF**36: Via 1mm, SloBloFP:Via 1mm, F.Cu at (244.6, 80.9)
- added REF**37: Via 1mm, SloBloFP:Via 1mm, F.Cu at (242.4, 79.1)
- added REF**38: Via 1mm, SloBloFP:Via 1mm, F.Cu at (239.7, 78.1)
- added REF**39: Via 1mm, SloBloFP:Via 1mm, F.Cu at (236.8, 77.9)
- added REF**4: Via 1mm, SloBloFP:Via 1mm, F.Cu at (234.5, 87.9)
- added REF**40: Via 1mm, SloBloFP:Via 1mm, F.Cu at (234.1, 78.5)
- added REF**41: Via 1mm, SloBloFP:Via 1mm, F.Cu at (231.5, 79.9)
- added REF**42: Via 1mm, SloBloFP:Via 1mm, F.Cu at (229.5, 81.9)
- added REF**43: Via 1mm, SloBloFP:Via 1mm, F.Cu at (228.1, 84.4)
- added REF**44: Via 1mm, SloBloFP:Via 1mm, F.Cu at (227.5, 87.2)
- added REF**45: Via 1mm, SloBloFP:Via 1mm, F.Cu at (227.7, 90.0)
- added REF**46: Via 1mm, SloBloFP:Via 1mm, F.Cu at (228.7, 92.7)
- added REF**47: Via 1mm, SloBloFP:Via 1mm, F.Cu at (230.4, 95.0)
- added REF**48: Via 1mm, SloBloFP:Via 1mm, F.Cu at (232.7, 96.7)
- added REF**49: Via 1mm, SloBloFP:Via 1mm, F.Cu at (235.3, 97.7)
- added REF**5: Via 1mm, SloBloFP:Via 1mm, F.Cu at (235.4, 90.0)
- added REF**50: Via 1mm, SloBloFP:Via 1mm, F.Cu at (238.2, 97.9)
- added REF**51: Via 1mm, SloBloFP:Via 1mm, F.Cu at (241.0, 97.3)
- added REF**52: Via 1mm, SloBloFP:Via 1mm, F.Cu at (243.5, 96.0)
- added REF**53: Via 1mm, SloBloFP:Via 1mm, F.Cu at (245.5, 94.0)
- added REF**54: Via 1mm, SloBloFP:Via 1mm, F.Cu at (246.9, 91.5)
- added REF**55: Via 1mm, SloBloFP:Via 1mm, F.Cu at (249.5, 84.4)
- added REF**56: Via 1mm, SloBloFP:Via 1mm, F.Cu at (248.4, 81.8)
- added REF**57: Via 1mm, SloBloFP:Via 1mm, F.Cu at (246.8, 79.6)
- added REF**58: Via 1mm, SloBloFP:Via 1mm, F.Cu at (244.7, 77.7)
- added REF**59: Via 1mm, SloBloFP:Via 1mm, F.Cu at (242.2, 76.4)
- added REF**6: Via 1mm, SloBloFP:Via 1mm, F.Cu at (237.5, 90.9)
- added REF**60: Via 1mm, SloBloFP:Via 1mm, F.Cu at (239.5, 75.6)
- added REF**61: Via 1mm, SloBloFP:Via 1mm, F.Cu at (236.8, 75.5)
- added REF**62: Via 1mm, SloBloFP:Via 1mm, F.Cu at (234.0, 76.0)
- added REF**63: Via 1mm, SloBloFP:Via 1mm, F.Cu at (231.4, 77.1)
- added REF**64: Via 1mm, SloBloFP:Via 1mm, F.Cu at (229.2, 78.7)
- added REF**65: Via 1mm, SloBloFP:Via 1mm, F.Cu at (227.3, 80.8)
- added REF**66: Via 1mm, SloBloFP:Via 1mm, F.Cu at (226.0, 83.2)
- added REF**67: Via 1mm, SloBloFP:Via 1mm, F.Cu at (225.2, 85.9)
- added REF**68: Via 1mm, SloBloFP:Via 1mm, F.Cu at (225.1, 88.7)
- added REF**69: Via 1mm, SloBloFP:Via 1mm, F.Cu at (225.6, 91.4)
- added REF**7: Via 1mm, SloBloFP:Via 1mm, F.Cu at (239.6, 90.0)
- added REF**70: Via 1mm, SloBloFP:Via 1mm, F.Cu at (226.7, 94.0)
- added REF**71: Via 1mm, SloBloFP:Via 1mm, F.Cu at (228.3, 96.3)
- added REF**72: Via 1mm, SloBloFP:Via 1mm, F.Cu at (230.4, 98.1)
- added REF**73: Via 1mm, SloBloFP:Via 1mm, F.Cu at (232.8, 99.5)
- added REF**74: Via 1mm, SloBloFP:Via 1mm, F.Cu at (235.5, 100.2)
- added REF**75: Via 1mm, SloBloFP:Via 1mm, F.Cu at (238.3, 100.3)
- added REF**76: Via 1mm, SloBloFP:Via 1mm, F.Cu at (241.0, 99.9)
- added REF**77: Via 1mm, SloBloFP:Via 1mm, F.Cu at (243.6, 98.8)
- added REF**78: Via 1mm, SloBloFP:Via 1mm, F.Cu at (245.9, 97.2)
- added REF**79: Via 1mm, SloBloFP:Via 1mm, F.Cu at (247.7, 95.1)
- added REF**8: Via 1mm, SloBloFP:Via 1mm, F.Cu at (240.8, 83.7)
- added REF**80: Via 1mm, SloBloFP:Via 1mm, F.Cu at (249.0, 92.6)
- added REF**81: Via 1mm, SloBloFP:Via 1mm, F.Cu at (249.8, 89.9)
- added REF**82: Via 1mm, SloBloFP:Via 1mm, F.Cu at (251.6, 82.7)
- added REF**83: Via 1mm, SloBloFP:Via 1mm, F.Cu at (250.4, 80.2)
- added REF**84: Via 1mm, SloBloFP:Via 1mm, F.Cu at (248.8, 78.0)
- added REF**85: Via 1mm, SloBloFP:Via 1mm, F.Cu at (246.8, 76.1)
- added REF**86: Via 1mm, SloBloFP:Via 1mm, F.Cu at (244.4, 74.6)
- added REF**87: Via 1mm, SloBloFP:Via 1mm, F.Cu at (241.9, 73.5)
- added REF**88: Via 1mm, SloBloFP:Via 1mm, F.Cu at (239.1, 73.0)
- added REF**89: Via 1mm, SloBloFP:Via 1mm, F.Cu at (236.4, 72.9)
- added REF**9: Via 1mm, SloBloFP:Via 1mm, F.Cu at (238.3, 82.6)
- added REF**90: Via 1mm, SloBloFP:Via 1mm, F.Cu at (233.6, 73.4)
- added REF**91: Via 1mm, SloBloFP:Via 1mm, F.Cu at (231.0, 74.4)
- added REF**92: Via 1mm, SloBloFP:Via 1mm, F.Cu at (228.6, 75.8)
- added REF**93: Via 1mm, SloBloFP:Via 1mm, F.Cu at (226.6, 77.6)
- added REF**94: Via 1mm, SloBloFP:Via 1mm, F.Cu at (224.8, 79.8)
- added REF**95: Via 1mm, SloBloFP:Via 1mm, F.Cu at (223.6, 82.3)
- added REF**96: Via 1mm, SloBloFP:Via 1mm, F.Cu at (222.8, 84.9)
- added REF**97: Via 1mm, SloBloFP:Via 1mm, F.Cu at (222.5, 87.7)
- added REF**98: Via 1mm, SloBloFP:Via 1mm, F.Cu at (222.7, 90.5)
- added REF**99: Via 1mm, SloBloFP:Via 1mm, F.Cu at (223.4, 93.1)
- moved H6 65.5 mm to (253.5, 171.9)
- moved REF** 65.5 mm to (216.0, 133.9)
- moved REF** 65.5 mm to (216.0, 161.4)
- moved REF** 65.5 mm to (103.5, 161.4)
- moved REF** 65.5 mm to (236.0, 133.9)
- moved REF** 65.5 mm to (93.5, 133.9)
- moved REF** 65.5 mm to (171.0, 161.4)
- moved REF** 65.5 mm to (128.5, 133.9)
- moved REF** 65.5 mm to (81.0, 161.4)
- moved REF** 65.5 mm to (193.5, 161.4)
- moved REF** 65.5 mm to (126.0, 161.4)
- moved REF** 65.5 mm to (236.0, 161.4)
- moved REF** 65.5 mm to (198.5, 134.7)
- moved REF** 65.5 mm to (148.5, 161.4)
- moved H1 65.5 mm to (42.5, 32.0)
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Other:
- board text removed: "SAW Amplitude"
- board text removed: "SAW Offset"
- board text removed: "SQUARE Amplitude"
- board text removed: "Square"
- board text removed: "Tracking"

Commit message: Algorithmic Speaker Grill added
Parts:
- removed the REF** at (242.5, 85.9)
- removed the REF** at (240.5, 87.9)
- removed the REF** at (237.5, 87.9)
- removed REF**1, REF**10, REF**100, REF**101, REF**102, REF**103, REF**104, REF**105, REF**106, REF**107, REF**108, REF**109, REF**11, REF**110, REF**111, REF**112, REF**113, REF**114, REF**115, REF**116, REF**117, REF**118, REF**119, REF**12, REF**120, REF**121, REF**122, REF**123, REF**124, REF**125, REF**126, REF**127, REF**128, REF**129, REF**13, REF**130, REF**131, REF**132, REF**133, REF**134, REF**135, REF**136, REF**137, REF**138, REF**139, REF**14, REF**140, REF**141, REF**142, REF**143, REF**144, REF**145, REF**146, REF**147, REF**148, REF**149, REF**15, REF**150, REF**151, REF**152, REF**153, REF**154, REF**155, REF**156, REF**157, REF**158, REF**159, REF**16, REF**160, REF**161, REF**162, REF**163, REF**164, REF**165, REF**166, REF**167, REF**168, REF**169, REF**17, REF**170, REF**171, REF**172, REF**173, REF**174, REF**175, REF**176, REF**177, REF**178, REF**179, REF**18 (x2), REF**180, REF**181, REF**182, REF**183, REF**184, REF**185, REF**186, REF**187, REF**188, REF**189, REF**19, REF**190, REF**191, REF**192, REF**193, REF**194, REF**195, REF**196, REF**197, REF**198, REF**199, REF**2, REF**20, REF**200 (x2), REF**201, REF**202, REF**203, REF**204, REF**205, REF**206, REF**207, REF**208, REF**209, REF**21, REF**210, REF**211, REF**212, REF**213, REF**214, REF**215, REF**216, REF**217, REF**218, REF**219, REF**22, REF**220, REF**221, REF**222, REF**223, REF**224, REF**225, REF**226, REF**227, REF**228, REF**229, REF**23, REF**230, REF**231, REF**232, REF**233, REF**234, REF**235, REF**236, REF**237, REF**238, REF**239, REF**24, REF**240, REF**241, REF**242, REF**243, REF**244, REF**245, REF**246, REF**247, REF**248, REF**249, REF**25, REF**250, REF**251, REF**252, REF**253, REF**254, REF**255, REF**26, REF**27, REF**28, REF**29, REF**3, REF**30, REF**31, REF**32, REF**33 (x6), REF**34, REF**35, REF**36, REF**37, REF**38, REF**39, REF**4, REF**40, REF**41, REF**42, REF**43, REF**44, REF**45, REF**46, REF**47, REF**48, REF**49, REF**5, REF**50, REF**51, REF**52, REF**53, REF**54, REF**55, REF**56, REF**57, REF**58, REF**59, REF**6, REF**60, REF**61, REF**62, REF**63, REF**64, REF**65, REF**66, REF**67, REF**68, REF**69, REF**7, REF**70, REF**71, REF**72, REF**73, REF**74, REF**75, REF**76, REF**77, REF**78, REF**79, REF**8, REF**80, REF**81, REF**82, REF**83, REF**84, REF**85, REF**86, REF**87, REF**88, REF**89, REF**9, REF**90, REF**91, REF**92, REF**93, REF**94, REF**95, REF**96, REF**97, REF**98, REF**99: Via 1mm, SloBloFP:Via 1mm
- added ?: , , F.Cu at (297.3, 115.8)
- added ?: , , F.Cu at (302.6, 122.2)
- added ?: , , F.Cu at (264.7, 126.5)
- added ?: , , F.Cu at (294.7, 123.0)
- added ?: , , F.Cu at (281.7, 142.6)
- added ?: , , F.Cu at (273.8, 143.6)
- added ?: , , F.Cu at (291.0, 132.3)
- added ?: , , F.Cu at (288.7, 155.5)
- added ?: , , F.Cu at (289.8, 141.8)
- added ?: , , F.Cu at (291.3, 136.1)
- added ?: , , F.Cu at (286.3, 135.3)
- added ?: , , F.Cu at (286.3, 123.3)
- added ?: , , F.Cu at (263.8, 142.1)
- added ?: , , F.Cu at (277.9, 130.9)
- added ?: , , F.Cu at (274.8, 136.7)
- added ?: , , F.Cu at (292.5, 137.8)
- added ?: , , F.Cu at (298.6, 145.2)
- added ?: , , F.Cu at (282.8, 128.5)
- added ?: , , F.Cu at (278.1, 150.3)
- added ?: , , F.Cu at (289.0, 152.7)
- added ?: , , F.Cu at (286.2, 142.2)
- added ?: , , F.Cu at (297.3, 128.0)
- added ?: , , F.Cu at (296.3, 138.2)
- added ?: , , F.Cu at (282.0, 146.5)
- added ?: , , F.Cu at (297.7, 118.5)
- added ?: , , F.Cu at (294.9, 130.3)
- added ?: , , F.Cu at (280.6, 155.2)
- added ?: , , F.Cu at (290.3, 122.2)
- added ?: , , F.Cu at (298.9, 125.5)
- added ?: , , F.Cu at (291.9, 145.9)
- added ?: , , F.Cu at (293.2, 141.8)
- added ?: , , F.Cu at (277.4, 123.0)
- added ?: , , F.Cu at (282.5, 157.2)
- added ?: , , F.Cu at (274.3, 154.6)
- added ?: , , F.Cu at (299.0, 129.6)
- added ?: , , F.Cu at (280.1, 125.8)
- added ?: , , F.Cu at (294.3, 114.7)
- added ?: , , F.Cu at (270.1, 130.0)
- added ?: , , F.Cu at (276.2, 152.7)
- added ?: , , F.Cu at (277.7, 147.3)
- added ?: , , F.Cu at (267.1, 128.3)
- added ?: , , F.Cu at (283.7, 120.9)
- added ?: , , F.Cu at (280.1, 116.2)
- added ?: , , F.Cu at (276.8, 137.3)
- added ?: , , F.Cu at (289.6, 139.8)
- added ?: , , F.Cu at (282.4, 135.4)
- added ?: , , F.Cu at (289.3, 143.8)
- added ?: , , F.Cu at (270.2, 137.3)
- added ?: , , F.Cu at (301.9, 124.8)
- added ?: , , F.Cu at (285.9, 128.1)
- added ?: , , F.Cu at (273.5, 129.9)
- added ?: , , F.Cu at (283.4, 112.3)
- added ?: , , F.Cu at (282.0, 122.3)
- added ?: , , F.Cu at (262.7, 134.1)
- added ?: , , F.Cu at (278.1, 111.9)
- added ?: , , F.Cu at (291.2, 114.1)
- added ?: , , F.Cu at (306.8, 136.0)
- added ?: , , F.Cu at (261.0, 136.3)
- added ?: , , F.Cu at (287.8, 119.3)
- added ?: , , F.Cu at (286.4, 153.9)
- added ?: , , F.Cu at (304.6, 140.9)
- added ?: , , F.Cu at (268.1, 139.5)
- added ?: , , F.Cu at (286.5, 111.7)
- added ?: , , F.Cu at (281.9, 152.6)
- added ?: , , F.Cu at (263.6, 137.0)
- added ?: , , F.Cu at (266.6, 141.9)
- added ?: , , F.Cu at (273.7, 123.5)
- added ?: , , F.Cu at (285.2, 144.0)
- added ?: , , F.Cu at (284.4, 117.2)
- added ?: , , F.Cu at (293.1, 112.1)
- added ?: , , F.Cu at (299.3, 142.6)
- added ?: , , F.Cu at (271.7, 142.6)
- added ?: , , F.Cu at (275.3, 113.5)
- added ?: , , F.Cu at (279.9, 147.1)
- added ?: , , F.Cu at (295.5, 126.7)
- added ?: , , F.Cu at (304.7, 124.6)
- added ?: , , F.Cu at (301.3, 144.8)
- added ?: , , F.Cu at (285.9, 137.2)
- added ?: , , F.Cu at (271.1, 153.6)
- added ?: , , F.Cu at (264.8, 132.3)
- added ?: , , F.Cu at (268.0, 117.8)
- added ?: , , F.Cu at (267.3, 130.9)
- added ?: , , F.Cu at (291.4, 154.0)
- added ?: , , F.Cu at (265.5, 134.9)
- added ?: , , F.Cu at (273.3, 152.0)
- added ?: , , F.Cu at (302.0, 136.5)
- added ?: , , F.Cu at (293.2, 149.2)
- added ?: , , F.Cu at (270.1, 125.3)
- added ?: , , F.Cu at (281.5, 138.6)
- added ?: , , F.Cu at (293.5, 125.9)
- added ?: , , F.Cu at (275.7, 133.2)
- added ?: , , F.Cu at (284.1, 138.5)
- added ?: , , F.Cu at (270.8, 122.9)
- added ?: , , F.Cu at (302.2, 139.2)
- added ?: , , F.Cu at (281.1, 110.6)
- added ?: , , F.Cu at (293.1, 129.4)
- added ?: , , F.Cu at (263.0, 144.8)
- added ?: , , F.Cu at (303.5, 132.1)
- added ?: , , F.Cu at (288.8, 137.7)
- added ?: , , F.Cu at (296.6, 140.3)
- added ?: , , F.Cu at (286.8, 116.6)
- added ?: , , F.Cu at (285.3, 114.3)
- added ?: , , F.Cu at (272.9, 149.3)
- added ?: , , F.Cu at (272.8, 115.5)
- added ?: , , F.Cu at (293.2, 139.8)
- added ?: , , F.Cu at (267.9, 133.3)
- added ?: , , F.Cu at (290.6, 147.8)
- added ?: , , F.Cu at (276.7, 125.0)
- added ?: , , F.Cu at (291.1, 129.1)
- added ?: , , F.Cu at (262.3, 127.8)
- added ?: , , F.Cu at (295.7, 144.9)
- added ?: , , F.Cu at (297.8, 133.3)
- added ?: , , F.Cu at (283.2, 141.0)
- added ?: , , F.Cu at (273.1, 127.8)
- added ?: , , F.Cu at (262.3, 131.0)
- added ?: , , F.Cu at (298.6, 150.3)
- added ?: , , F.Cu at (300.7, 127.4)
- added ?: , , F.Cu at (289.8, 111.7)
- added ?: , , F.Cu at (275.3, 147.1)
- added ?: , , F.Cu at (280.2, 119.6)
- added ?: , , F.Cu at (291.4, 125.6)
- added ?: , , F.Cu at (274.7, 121.4)
- added ?: , , F.Cu at (297.4, 147.7)
- added ?: , , F.Cu at (270.7, 132.1)
- added ?: , , F.Cu at (295.2, 120.1)
- added ?: , , F.Cu at (286.5, 140.0)
- added ?: , , F.Cu at (292.5, 122.4)
- added ?: , , F.Cu at (285.6, 119.9)
- added ?: , , F.Cu at (306.9, 139.3)
- added ?: , , F.Cu at (288.9, 129.4)
- added ?: , , F.Cu at (304.0, 144.0)
- added ?: , , F.Cu at (280.0, 132.6)
- added ?: , , F.Cu at (282.1, 118.2)
- added ?: , , F.Cu at (306.4, 127.4)
- added ?: , , F.Cu at (297.6, 121.3)
- added ?: , , F.Cu at (262.2, 139.3)
- added ?: , , F.Cu at (296.5, 131.6)
- added ?: , , F.Cu at (275.9, 144.0)
- added ?: , , F.Cu at (279.1, 152.9)
- added ?: , , F.Cu at (276.5, 127.0)
- added ?: , , F.Cu at (292.7, 119.4)
- added ?: , , F.Cu at (277.5, 140.6)
- added ?: , , F.Cu at (291.3, 151.1)
- added ?: , , F.Cu at (275.5, 140.5)
- added ?: , , F.Cu at (282.9, 149.5)
- added ?: , , F.Cu at (301.4, 134.0)
- added ?: , , F.Cu at (283.7, 145.4)
- added ?: , , F.Cu at (289.4, 125.8)
- added ?: , , F.Cu at (280.7, 134.6)
- added ?: , , F.Cu at (287.5, 126.6)
- added ?: , , F.Cu at (289.4, 134.8)
- added ?: , , F.Cu at (275.5, 116.3)
- added ?: , , F.Cu at (265.3, 147.2)
- added ?: , , F.Cu at (284.5, 131.0)
- added ?: , , F.Cu at (299.9, 122.8)
- added ?: , , F.Cu at (273.0, 146.5)
- added ?: , , F.Cu at (306.2, 132.9)
- added ?: , , F.Cu at (270.5, 150.9)
- added ?: , , F.Cu at (277.8, 114.6)
- added ?: , , F.Cu at (268.8, 135.5)
- added ?: , , F.Cu at (273.6, 139.9)
- added ?: , , F.Cu at (280.0, 143.6)
- added ?: , , F.Cu at (262.8, 124.6)
- added ?: , , F.Cu at (292.2, 116.6)
- added ?: , , F.Cu at (288.4, 132.3)
- added ?: , , F.Cu at (277.6, 134.3)
- added ?: , , F.Cu at (296.9, 124.0)
- added ?: , , F.Cu at (279.6, 140.0)
- added ?: , , F.Cu at (274.3, 131.7)
- added ?: , , F.Cu at (294.1, 154.8)
- added ?: , , F.Cu at (264.5, 129.4)
- added ?: , , F.Cu at (273.5, 118.3)
- added ?: , , F.Cu at (268.0, 122.9)
- added ?: , , F.Cu at (288.9, 149.5)
- added ?: , , F.Cu at (305.1, 129.9)
- added ?: , , F.Cu at (277.4, 155.2)
- added ?: , , F.Cu at (280.8, 123.9)
- added ?: , , F.Cu at (276.8, 129.0)
- added ?: , , F.Cu at (302.9, 147.1)
- added ?: , , F.Cu at (273.1, 135.6)
- added ?: , , F.Cu at (304.6, 137.8)
- added ?: , , F.Cu at (269.9, 127.7)
- added ?: , , F.Cu at (296.4, 142.6)
- added ?: , , F.Cu at (270.7, 145.4)
- added ?: , , F.Cu at (302.3, 129.6)
- added ?: , , F.Cu at (270.3, 148.1)
- added ?: , , F.Cu at (286.8, 147.2)
- added ?: , , F.Cu at (290.2, 119.2)
- added ?: , , F.Cu at (299.4, 137.6)
- added ?: , , F.Cu at (265.7, 144.5)
- added ?: , , F.Cu at (278.6, 121.2)
- added ?: , , F.Cu at (270.1, 115.2)
- added ?: , , F.Cu at (283.4, 126.2)
- added ?: , , F.Cu at (304.3, 134.9)
- added ?: , , F.Cu at (283.5, 132.6)
- added ?: , , F.Cu at (280.7, 130.3)
- added ?: , , F.Cu at (288.2, 113.9)
- added ?: , , F.Cu at (284.0, 134.0)
- added ?: , , F.Cu at (292.8, 143.9)
- added ?: , , F.Cu at (285.7, 156.6)
- added ?: , , F.Cu at (280.6, 150.1)
- added ?: , , F.Cu at (293.8, 152.1)
- added ?: , , F.Cu at (282.6, 115.0)
- added ?: , , F.Cu at (283.6, 154.8)
- added ?: , , F.Cu at (280.5, 113.2)
- added ?: , , F.Cu at (294.5, 134.5)
- added ?: , , F.Cu at (284.7, 124.5)
- added ?: , , F.Cu at (302.0, 142.0)
- added ?: , , F.Cu at (265.3, 123.5)
- added ?: , , F.Cu at (293.0, 133.2)
- added ?: , , F.Cu at (299.6, 140.1)
- added ?: , , F.Cu at (289.5, 116.4)
- added ?: , , F.Cu at (273.2, 125.7)
- added ?: , , F.Cu at (286.8, 150.9)
- added ?: , , F.Cu at (267.8, 149.3)
- added ?: , , F.Cu at (286.5, 130.9)
- added ?: , , F.Cu at (300.2, 147.6)
- added ?: , , F.Cu at (288.3, 145.6)
- added ?: , , F.Cu at (295.0, 117.3)
- added ?: , , F.Cu at (288.2, 122.6)
- added ?: , , F.Cu at (300.2, 120.1)
- added ?: , , F.Cu at (271.8, 138.8)
- added ?: , , F.Cu at (298.8, 135.4)
- added ?: , , F.Cu at (301.4, 150.0)
- added ?: , , F.Cu at (269.8, 141.2)
- added ?: , , F.Cu at (300.3, 131.6)
- added ?: , , F.Cu at (278.0, 117.7)
- added ?: , , F.Cu at (272.0, 120.5)
- added ?: , , F.Cu at (295.8, 150.0)
- added ?: , , F.Cu at (267.9, 146.5)
- added ?: , , F.Cu at (296.5, 152.7)
- added ?: , , F.Cu at (300.1, 117.3)
- added ?: , , F.Cu at (275.5, 150.0)
- added ?: , , F.Cu at (276.1, 119.4)
- added ?: , , F.Cu at (266.6, 137.3)
- added ?: , , F.Cu at (265.0, 139.6)
- added ?: , , F.Cu at (278.0, 144.1)
- added ?: , , F.Cu at (294.7, 147.1)
- added ?: , , F.Cu at (285.0, 148.5)
- added ?: , , F.Cu at (268.5, 143.8)
- added ?: , , F.Cu at (284.5, 151.9)
- added ?: , , F.Cu at (295.6, 136.2)
- added ?: , , F.Cu at (267.3, 125.6)
- added ?: , , F.Cu at (269.2, 120.3)
- added ?: , , F.Cu at (303.7, 127.2)
- added ?: , , F.Cu at (266.4, 120.6)
- added ?: , , F.Cu at (279.1, 137.1)
- added ?: , , F.Cu at (271.7, 134.0)
- added ?: , , F.Cu at (279.9, 127.9)
- added ?: , , F.Cu at (270.8, 117.8)
- added J1: PJ398SM, SloBlo:Thonkiconn_PJ398SM, F.Cu at (264.3, 90.7)
- added J2: PJ398SM, SloBlo:Thonkiconn_PJ398SM, F.Cu at (280.0, 90.8)
- added J3: PJ398SM, SloBlo:Thonkiconn_PJ398SM, F.Cu at (298.8, 90.8)
- added LS1: LSM-50M/NO-B 8R (<32R) 1W, SloBlo:LSM-50M NO-B, F.Cu at (284.0, 134.0)
- added RGB_Pot1: TC002-N11AS2XT-RGB, SloBlo:TC002-N11AS2XT-RGB, F.Cu at (262.5, 180.0)
- added RGB_Pot2: TC002-N11AS2XT-RGB, SloBlo:TC002-N11AS2XT-RGB, F.Cu at (105.0, 207.4)
- added RGB_Pot3: TC002-N11AS2XT-RGB, SloBlo:TC002-N11AS2XT-RGB, F.Cu at (127.5, 207.4)
- added RGB_Pot4: TC002-N11AS2XT-RGB, SloBlo:TC002-N11AS2XT-RGB, F.Cu at (150.0, 207.5)
- added RGB_Pot5: TC002-N11AS2XT-RGB, SloBlo:TC002-N11AS2XT-RGB, F.Cu at (172.5, 207.5)
- added RGB_Pot6: TC002-N11AS2XT-RGB, SloBlo:TC002-N11AS2XT-RGB, F.Cu at (195.0, 207.5)
- added RGB_Pot7: TC002-N11AS2XT-RGB, SloBlo:TC002-N11AS2XT-RGB, F.Cu at (217.5, 207.5)
- added RGB_Pot8: TC002-N11AS2XT-RGB, SloBlo:TC002-N11AS2XT-RGB, F.Cu at (240.0, 207.5)
- added RGB_Pot9: TC002-N11AS2XT-RGB, SloBlo:TC002-N11AS2XT-RGB, F.Cu at (262.5, 207.5)
- added RV1: 1K, SloBlo:Potentiometer_Bourns_3296W_Vertical, F.Cu at (230.5, 75.0)
- added RV10: 100K, SloBlo:RV141F-40-20BL, F.Cu at (174.9, 120.0)
- added RV11: 100k, SloBlo:RV141F-40-20BL, F.Cu at (209.9, 120.0)
- added RV12: 100, SloBlo:Potentiometer_Bourns_3296W_Vertical, F.Cu at (90.5, 131.2)
- added RV13: 100K, SloBlo:Alpha_RD901F, F.Cu at (104.9, 150.0)
- added RV14: 100K, SloBlo:Alpha_RD901F, F.Cu at (139.9, 150.0)
- added RV15: 100K, SloBlo:Potentiometer_Bourns_3296W_Vertical, F.Cu at (90.5, 142.2)
- added RV16: 100K, SloBlo:Potentiometer_Bourns_3296W_Vertical, F.Cu at (90.5, 153.2)
- added RV17: 100K, SloBlo:Potentiometer_Bourns_3296W_Vertical, F.Cu at (90.5, 164.2)
- added RV18: 100K, SloBlo:Alpha_RD901F, F.Cu at (105.0, 180.0)
- added RV19: 100K, SloBlo:Alpha_RD901F, F.Cu at (140.0, 180.0)
- added RV2: 100, SloBlo:Potentiometer_Bourns_3296W_Vertical, F.Cu at (117.0, 81.4)
- added RV20: 100K, SloBlo:Alpha_RD901F, F.Cu at (175.0, 180.0)
- added RV21: 10K, SloBlo:Alpha_RD901F, F.Cu at (282.5, 180.0)
- added RV22: 100K, SloBlo:Alpha_RD901F, F.Cu at (245.0, 180.8)
- added RV3: 100K, SloBlo:Alpha_RD901F, F.Cu at (244.9, 90.0)
- added RV4: 10K, SloBlo:RV141F-40-20BL, F.Cu at (104.9, 90.0)
- added RV5: 100K, SloBlo:RV141F-40-20BL, F.Cu at (139.9, 90.0)
- added RV6: 100K, SloBlo:RV141F-40-20BL, F.Cu at (174.9, 90.0)
- added RV7: 100K, SloBlo:RV141F-40-20BL, F.Cu at (209.9, 90.0)
- added RV8: 100K, SloBlo:Alpha_RD901F, F.Cu at (244.9, 120.0)
- added RV9: 10K, SloBlo:RV141F-40-20BL, F.Cu at (139.9, 120.0)
- added SW1: SW_SPDT, SloBlo:SW_Toggle_MS500C, F.Cu at (104.9, 120.0)
- added SW2: SW_SPST, SloBlo:SW_Toggle_MS500C, F.Cu at (174.9, 150.0)
- added SW3: SW_SPDT, SloBlo:SW_Toggle_MS500C, F.Cu at (209.9, 150.0)
- added SW4: SW_SPDT, SloBlo:SW_Toggle_MS500C, F.Cu at (244.9, 150.0)
- added SW6: SW_Push, SloBlo:E-Switch_TL1105SP, F.Cu at (282.5, 207.5)
- moved H6 65.5 mm to (300.0, 217.9)
- moved REF** 65.5 mm to (262.5, 180.0)
- moved REF** 65.5 mm to (262.5, 207.5)
- moved REF** 65.5 mm to (150.0, 207.5)
- moved REF** 65.5 mm to (282.5, 180.0)
- moved REF** 65.5 mm to (140.0, 180.0)
- moved REF** 65.5 mm to (217.5, 207.5)
- moved REF** 65.5 mm to (175.0, 180.0)
- moved REF** 65.5 mm to (127.5, 207.4)
- moved REF** 65.5 mm to (240.0, 207.5)
- moved REF** 65.5 mm to (172.5, 207.5)
- moved REF** 65.5 mm to (282.5, 207.5)
- moved REF** 65.5 mm to (245.0, 180.8)
- moved REF** 65.5 mm to (195.0, 207.5)
- moved H1 65.5 mm to (89.0, 78.0)
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Other:
- board text added: "SAW Amplitude"
- board text added: "SAW Offset"
- board text added: "SQUARE Amplitude"
- board text added: "Square"
- board text added: "Tracking"
