File: hardware/KiCad/LivSynth_0v2/IO.kicad_sch (KiCad schematic)
At the start: 95 parts, among them J1 PJ398SM, J10 Jumper, J11 Jumper, J2 PJ398SM, J20 IDC, J3 PJ398SM, J4 IDC, Q3 2N3904, Q4 2N3904, SW5 SW_Push, U10 74HC165, U11 PCA9685PW, U12 PCA9685PW, U13 74HC165, U2 LM386

Commit message: Before fixing HW issues
Parts:
- R34: value 20K -> 4K7
Other:
- note added: "7/,4 = (100K+R)/R <=> R = 100K/(7/,4 - 1) = 6,06K"
- note added: "7Vpp"
- note added: "8Vpp max"
- note added: "8Vpp/20 = 0,4Vpp max"
Changed lines of the file:
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@@
+    (effects (font (size 1.27 1.27)) (justify left bottom))
+  )
+  (text "8Vpp/20 =\n0,4Vpp max" (at 320.04 68.58 0)
     (effects (font (size 1.27 1.27)) (justify left bottom))
   )
@@
     (effects (font (size 1.27 1.27)) (justify left bottom))
   )
+  (text "7/,4 = (100K+R)/R\n<=> R = 100K/(7/,4 - 1) = 6,06K" (at 269.24 69.85 0)
+    (effects (font (size 1.27 1.27)) (justify left bottom))
+  )
   (text "Address 0x02" (at 133.985 22.86 0)
     (effects (font (size 1.27 1.27)) (justify left bottom))
@@
   )
   (text "External" (at 384.81 60.96 0)
+    (effects (font (size 1.27 1.27)) (justify left bottom))
+  )
+  (text "8Vpp max" (at 345.44 64.77 0)
+    (effects (font (size 1.27 1.27)) (justify left bottom))
+  )
+  (text "7Vpp" (at 316.23 30.48 0)
     (effects (font (size 1.27 1.27)) (justify left bottom))
   )
@@
   (symbol (lib_id "Device:R") (at 309.245 70.485 0) (unit 1)
     (in_bom yes) (on_board yes) (fields_autoplaced)
-    (property "Reference" "R34" (id 0) (at 311.785 69.2149 0)
-      (effects (font (size 1.27 1.27)) (justify left))
-    )
-    (property "Value" "20K" (id 1) (at 311.785 71.7549 0)
-      (effects (font (size 1.27 1.27)) (justify left))
-    )
+    (property "Reference" "R34" (id 0) (at 311.15 69.2149 0)
+      (effects (font (size 1.27 1.27)) (justify left))
+    )
+    (property "Value" "4K7" (id 1) (at 311.15 71.7549 0)
+      (effects (font (size 1.27 1.27)) (justify left))
+    )

Commit message: Analog redesign:  - Power: Add voltage and current test points  - MCU: use PA11/PA12 for USB DFU interface  - MCU: add NRST reset switch  - Slew: increase portamento cap  - VCO: invert trim pots  - VCF: let resonance kick in earlier  - VCF: invert pots  - VCA: invert trim pot  - EG: full redesign, properly referencing VGND now  - LFO: R61 = 51K  - ModMatrix: add EG attenuverters  - IO: invert pots  - IO: limit output gain for 1W speaker  - IO: connect BTN_SHIFT in gap free order to SR
Parts:
- R34: value 4K7 -> 6K2
Connections:
- net +3.3VA: now also RV1.3, RV22.3; no longer RV1.1, RV22.1
- net BTN_SHIFT: now also U10.12 (D1); no longer U10.6 (D7)
- net GND: now also RV1.1, RV22.1, U10.13 (D2), U10.14 (D3), U10.3 (D4), U10.4 (D5), U10.5 (D6), U10.6 (D7); no longer RV1.3, RV22.3
- no-connect marks 30 -> 24
Other:
- note added: "P = U * I = U^2 / R <=> U = SQRT(P * R) = SQRT(1W * 8R) = 2,83V Upp = 2 * 2,83V * SQRT(2) = 8Vpp max"
Changed lines of the file:
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@@
   (junction (at 128.905 137.16) (diameter 0) (color 0 0 0 0)
   )
+  (junction (at 223.52 58.42) (diameter 0) (color 0 0 0 0)
+  )
   (junction (at 242.57 135.89) (diameter 0) (color 0 0 0 0)
   )
@@
   (junction (at 193.04 94.615) (diameter 0) (color 0 0 0 0)
   )
+  (junction (at 223.52 50.8) (diameter 0) (color 0 0 0 0)
+  )
   (junction (at 81.915 95.25) (diameter 0) (color 0 0 0 0)
   )
@@
   (junction (at 309.245 64.135) (diameter 0) (color 0 0 0 0)
   )
+  (junction (at 223.52 48.26) (diameter 0) (color 0 0 0 0)
+  )
   (junction (at 34.29 137.16) (diameter 0) (color 0 0 0 0)
   )
   (junction (at 108.585 69.215) (diameter 0) (color 0 0 0 0)
   )
+  (junction (at 223.52 53.34) (diameter 0) (color 0 0 0 0)
+  )
+  (junction (at 223.52 55.88) (diameter 0) (color 0 0 0 0)
+  )
   (no_connect (at 234.315 139.065))
   (no_connect (at 224.155 139.065))
@@
   (no_connect (at 203.835 40.64))
   (no_connect (at 80.01 71.755))
-  (no_connect (at 225.425 43.18))
   (no_connect (at 31.75 97.79))
   (no_connect (at 41.91 97.79))
   (no_connect (at 126.365 139.7))
   (no_connect (at 188.595 186.69))
-  (no_connect (at 225.425 55.88))
   (no_connect (at 89.535 97.79))
-  (no_connect (at 225.425 48.26))
   (no_connect (at 184.785 97.79))
   (no_connect (at 250.825 40.64))
   (no_connect (at 31.75 139.7))
   (no_connect (at 136.525 139.7))
-  (no_connect (at 225.425 50.8))
-  (no_connect (at 225.425 53.34))
   (no_connect (at 184.785 139.065))
   (no_connect (at 41.91 139.7))
-  (no_connect (at 225.425 45.72))
   (no_connect (at 146.05 71.755))
   (no_connect (at 126.365 186.69))
@@
     (stroke (width 0) (type default) (color 0 0 0 0))
   )
-  (wire (pts (xy 220.345 58.42) (xy 225.425 58.42))
+  (wire (pts (xy 220.345 43.18) (xy 225.425 43.18))
     (stroke (width 0) (type default) (color 0 0 0 0))
   )
@@
     (stroke (width 0) (type default) (color 0 0 0 0))
   )
+  (wire (pts (xy 223.52 50.8) (xy 223.52 48.26))
+    (stroke (width 0) (type default) (color 0 0 0 0))
+  )
   (wire (pts (xy 240.665 154.305) (xy 242.57 154.305))
     (stroke (width 0) (type default) (color 0 0 0 0))
@@
     (stroke (width 0) (type default) (color 0 0 0 0))
   )
+  (wire (pts (xy 223.52 48.26) (xy 223.52 45.72))
+    (stroke (width 0) (type default) (color 0 0 0 0))
+  )
   (wire (pts (xy 42.545 64.135) (xy 44.45 64.135))
     (stroke (width 0) (type default) (color 0 0 0 0))
@@
     (stroke (width 0) (type default) (color 0 0 0 0))
   )
+  (wire (pts (xy 223.52 53.34) (xy 225.425 53.34))
+    (stroke (width 0) (type default) (color 0 0 0 0))
+  )
   (wire (pts (xy 193.04 92.075) (xy 193.04 94.615))
     (stroke (width 0) (type default) (color 0 0 0 0))
@@
     (stroke (width 0) (type default) (color 0 0 0 0))
   )
+  (wire (pts (xy 223.52 48.26) (xy 225.425 48.26))
+    (stroke (width 0) (type default) (color 0 0 0 0))
+  )
   (wire (pts (xy 86.995 94.615) (xy 97.79 94.615))
     (stroke (width 0) (type default) (color 0 0 0 0))
@@
     (stroke (width 0) (type default) (color 0 0 0 0))
   )
+  (wire (pts (xy 223.52 50.8) (xy 225.425 50.8))
+    (stroke (width 0) (type default) (color 0 0 0 0))
+  )
   (wire (pts (xy 144.78 162.56) (xy 144.78 160.02))
     (stroke (width 0) (type default) (color 0 0 0 0))
@@
     (stroke (width 0) (type default) (color 0 0 0 0))
   )
+  (wire (pts (xy 223.52 58.42) (xy 223.52 55.88))
+    (stroke (width 0) (type default) (color 0 0 0 0))
+  )
   (wire (pts (xy 107.95 36.195) (xy 110.49 36.195))
     (stroke (width 0) (type default) (color 0 0 0 0))
@@
     (stroke (width 0) (type default) (color 0 0 0 0))
   )
+  (wire (pts (xy 223.52 55.88) (xy 225.425 55.88))
+    (stroke (width 0) (type default) (color 0 0 0 0))
+  )
   (wire (pts (xy 164.465 100.33) (xy 166.37 100.33))
     (stroke (width 0) (type default) (color 0 0 0 0))
@@
     (stroke (width 0) (type default) (color 0 0 0 0))
   )
+  (wire (pts (xy 223.52 55.88) (xy 223.52 53.34))
+    (stroke (width 0) (type default) (color 0 0 0 0))
+  )
   (wire (pts (xy 97.79 120.65) (xy 97.79 118.11))
     (stroke (width 0) (type default) (color 0 0 0 0))
@@
     (stroke (width 0) (type default) (color 0 0 0 0))
   )
+  (wire (pts (xy 223.52 53.34) (xy 223.52 50.8))
+    (stroke (width 0) (type default) (color 0 0 0 0))
+  )
   (wire (pts (xy 227.33 26.035) (xy 227.33 25.4))
     (stroke (width 0) (type default) (color 0 0 0 0))
@@
     (stroke (width 0) (type default) (color 0 0 0 0))
   )
+  (wire (pts (xy 223.52 59.055) (xy 223.52 58.42))
+    (stroke (width 0) (type default) (color 0 0 0 0))
+  )
   (wire (pts (xy 146.05 53.975) (xy 149.86 53.975))
     (stroke (width 0) (type default) (color 0 0 0 0))
@@
     (stroke (width 0) (type default) (color 0 0 0 0))
   )
+  (wire (pts (xy 223.52 45.72) (xy 225.425 45.72))
+    (stroke (width 0) (type default) (color 0 0 0 0))
+  )
   (wire (pts (xy 41.91 37.465) (xy 44.45 37.465))
     (stroke (width 0) (type default) (color 0 0 0 0))
@@
     (stroke (width 0) (type default) (color 0 0 0 0))
   )
+  (wire (pts (xy 223.52 58.42) (xy 225.425 58.42))
+    (stroke (width 0) (type default) (color 0 0 0 0))
+  )
   (wire (pts (xy 81.915 134.62) (xy 81.915 137.16))
     (stroke (width 0) (type default) (color 0 0 0 0))
@@
     (effects (font (size 1.27 1.27)) (justify left bottom))
   )
+  (text "P = U * I = U^2 / R\n<=> U = SQRT(P * R)\n  = SQRT(1W * 8R)\n  = 2,83V\nUpp = 2 * 2,83V * SQRT(2) = 8Vpp max"
+    (at 365.125 93.98 0)
+    (effects (font (size 1.27 1.27)) (justify left bottom))
+  )
   (text "7Vpp" (at 316.23 30.48 0)
     (effects (font (size 1.27 1.27)) (justify left bottom))
@@
     (effects (font (size 1.27 1.27)) (justify right bottom))
   )
-  (label "BTN_SHIFT" (at 220.345 58.42 180)
+  (label "BTN_SHIFT" (at 220.345 43.18 180)
     (effects (font (size 1.27 1.27)) (justify right bottom))
   )
@@
       (effects (font (size 1.27 1.27)) (justify left))
     )
-    (property "Value" "4K7" (id 1) (at 311.15 71.7549 0)
+    (property "Value" "6K2" (id 1) (at 311.15 71.7549 0)
       (effects (font (size 1.27 1.27)) (justify left))
     )
@@
     (pin "1")
   )
+  (symbol (lib_id "power:GND") (at 223.52 59.055 0) (unit 1)
+    (in_bom yes) (on_board yes) (fields_autoplaced)
+    (property "Reference" "#PWR?" (id 0) (at 223.52 65.405 0)
+      (effects (font (size 1.27 1.27)) hide)
+    )
+    (property "Value" "GND" (id 1) (at 223.52 63.5 0)
+      (effects (font (size 1.27 1.27)) hide)
+    )
+    (property "Footprint" "" (id 2) (at 223.52 59.055 0)
+      (effects (font (size 1.27 1.27)) hide)
+    )
+    (property "Datasheet" "" (id 3) (at 223.52 59.055 0)
+      (effects (font (size 1.27 1.27)) hide)
+    )
+    (pin "1")
+  )
   (symbol (lib_id "power:GND") (at 376.555 42.545 0) (unit 1)
     (in_bom yes) (on_board yes) (fields_autoplaced)
@@
     (pin "1")
   )
-  (symbol (lib_id "Device:R_Potentiometer") (at 56.515 184.15 0) (unit 1)
+  (symbol (lib_id "Device:R_Potentiometer") (at 56.515 184.15 0) (mirror x) (unit 1)
     (in_bom yes) (on_board yes) (fields_autoplaced)
     (property "Reference" "RV22" (id 0) (at 54.61 182.8799 0)
@@
     (pin "1")
   )
-  (symbol (lib_id "Device:R_Potentiometer") (at 24.765 184.15 0) (unit 1)
+  (symbol (lib_id "Device:R_Potentiometer") (at 24.765 184.15 0) (mirror x) (unit 1)
     (in_bom yes) (on_board yes) (fields_autoplaced)
     (property "Reference" "RV1" (id 0) (at 22.86 182.8799 0)

Commit message: Analog Redesign:  - Power: Build ververse polarity protection using P-Mosfet and Zener Diode      - (https://www.youtube.com/watch?v=Ltx4vovY5Z4 - 1:28)  - Power: Build adjustable buck regulator for 8-9V stable voltage source  - PCB: Add location for order number ("JLCJLCJLCJLC")  - General: Add Tooling Holes for PCB assembly  - PCB: check frontend component layout for symmetry  - VCF: fix sound issues  - PCB: Add SloBlo icon  - PCB: Add switch labels to front side  - EG: test new design  - MCU: Add some debug pins
Parts:
- U10, U13: LCSC (none) -> C7334
- U11, U12: LCSC (none) -> C2688894
Changed lines of the file:
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@@
+      (effects (font (size 1.27 1.27)) hide)
+    )
+    (property "LCSC" "C2688894" (id 4) (at 62.23 51.435 0)
       (effects (font (size 1.27 1.27)) hide)
     )
@@
       (effects (font (size 1.27 1.27)) hide)
     )
+    (property "LCSC" "C7334" (id 4) (at 238.125 53.34 0)
+      (effects (font (size 1.27 1.27)) hide)
+    )
     (pin "1")
     (pin "10")
@@
   (symbol (lib_id "power:GND") (at 223.52 59.055 0) (unit 1)
     (in_bom yes) (on_board yes) (fields_autoplaced)
-    (property "Reference" "#PWR?" (id 0) (at 223.52 65.405 0)
+    (property "Reference" "#PWR0145" (id 0) (at 223.52 65.405 0)
       (effects (font (size 1.27 1.27)) hide)
     )
@@
     )
     (property "Datasheet" "http://www.nxp.com/documents/data_sheet/PCA9685.pdf" (id 3) (at 118.11 33.655 0)
+      (effects (font (size 1.27 1.27)) hide)
+    )
+    (property "LCSC" "C2688894" (id 4) (at 128.27 51.435 0)
       (effects (font (size 1.27 1.27)) hide)
     )
@@
       (effects (font (size 1.27 1.27)) hide)
     )
+    (property "LCSC" "C7334" (id 4) (at 191.135 53.34 0)
+      (effects (font (size 1.27 1.27)) hide)
+    )
