File: hardware/Mainboard/IO.kicad_sch (KiCad schematic)
At the start: 95 parts, among them J1 PJ398SM, J13 Jumper, J14 Jumper, J2 PJ398SM, J20 IDC, J3 PJ398SM, J4 IDC, Q6 2N3904, Q7 2N3904, SW6 SW_Push, U10 PCA9685PW, U11 PCA9685PW, U13 74HC165, U14 74HC165, U3 LM386

Commit message: exxclude pre-assebled and not required components from BOM
Parts:
- J14, J4: now left out of the parts list
Changed lines of the file:
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@@
   )
   (symbol (lib_id "Connector:Conn_01x02_Male") (at 338.455 80.645 90) (unit 1)
-    (in_bom yes) (on_board yes) (dnp no)
+    (in_bom no) (on_board yes) (dnp no)
     (property "Reference" "J14" (at 342.265 80.01 90)
       (effects (font (size 1.27 1.27)) (justify right))
@@
   )
   (symbol (lib_id "Connector:Conn_01x02_Male") (at 370.84 66.675 0) (mirror y) (unit 1)
-    (in_bom yes) (on_board yes) (dnp no)
+    (in_bom no) (on_board yes) (dnp no)
     (property "Reference" "J4" (at 365.76 60.325 0)
       (effects (font (size 1.27 1.27)) (justify right))
