File: hardware/Mainboard/Power.kicad_sch (KiCad schematic)
At the start: 61 parts, among them J12 VGND, J201 Test Points, J24 3V3, J25 9V, J7 Barrel_Jack_Switch, Q3 AO3401A, SW7 SW_SPDT, U1 TL074, U12 TPS63070, U2 TL074, U4 TL074, U5 TL074, U6 TL074, U7 LM13700, U8 LM1117-3.3

Commit message: exxclude pre-assebled and not required components from BOM
Parts:
- C53, C54, C55, C56, C57, C60, C63, C64, D4, J201, L1, Q3, R115, R94, R95, R96, U12: now left out of the parts list
Changed lines of the file:
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@@
   )
   (symbol (lib_id "Device:C") (at 159.385 80.645 0) (unit 1)
-    (in_bom yes) (on_board yes) (dnp no)
+    (in_bom no) (on_board yes) (dnp no)
     (property "Reference" "C54" (at 162.56 78.74 0)
       (effects (font (size 1.27 1.27)) (justify left))
@@
   )
   (symbol (lib_id "Device:C") (at 41.275 80.645 0) (unit 1)
-    (in_bom yes) (on_board yes) (dnp no) (fields_autoplaced)
+    (in_bom no) (on_board yes) (dnp no) (fields_autoplaced)
     (property "Reference" "C63" (at 44.45 78.4859 0)
       (effects (font (size 1.27 1.27)) (justify left))
@@
   )
   (symbol (lib_id "Device:D_Zener_Small") (at 91.44 29.21 270) (unit 1)
-    (in_bom yes) (on_board yes) (dnp no) (fields_autoplaced)
+    (in_bom no) (on_board yes) (dnp no) (fields_autoplaced)
     (property "Reference" "D4" (at 93.345 27.9399 90)
       (effects (font (size 1.27 1.27)) (justify left))
@@
   )
   (symbol (lib_id "SloBlo:TPS63070x") (at 94.615 91.44 0) (unit 1)
-    (in_bom yes) (on_board yes) (dnp no)
+    (in_bom no) (on_board yes) (dnp no)
     (property "Reference" "U12" (at 86.36 118.745 0)
       (effects (font (size 1.524 1.524)))
@@
   )
   (symbol (lib_id "Device:R_Small") (at 64.135 81.28 0) (unit 1)
-    (in_bom yes) (on_board yes) (dnp no) (fields_autoplaced)
+    (in_bom no) (on_board yes) (dnp no) (fields_autoplaced)
     (property "Reference" "R115" (at 67.31 80.0099 0)
       (effects (font (size 1.27 1.27)) (justify left))
@@
   )
   (symbol (lib_id "Device:C") (at 29.845 80.645 0) (unit 1)
-    (in_bom yes) (on_board yes) (dnp no) (fields_autoplaced)
+    (in_bom no) (on_board yes) (dnp no) (fields_autoplaced)
     (property "Reference" "C64" (at 33.02 78.4859 0)
       (effects (font (size 1.27 1.27)) (justify left))
@@
   )
   (symbol (lib_id "Transistor_FET:AO3401A") (at 83.185 27.305 90) (unit 1)
-    (in_bom yes) (on_board yes) (dnp no) (fields_autoplaced)
+    (in_bom no) (on_board yes) (dnp no) (fields_autoplaced)
     (property "Reference" "Q3" (at 83.185 17.145 90)
       (effects (font (size 1.27 1.27)))
@@
   )
   (symbol (lib_id "Device:C") (at 170.18 80.645 0) (unit 1)
-    (in_bom yes) (on_board yes) (dnp no)
+    (in_bom no) (on_board yes) (dnp no)
     (property "Reference" "C53" (at 173.355 78.74 0)
       (effects (font (size 1.27 1.27)) (justify left))
@@
   )
   (symbol (lib_id "Device:L") (at 94.615 61.595 90) (unit 1)
-    (in_bom yes) (on_board yes) (dnp no) (fields_autoplaced)
+    (in_bom no) (on_board yes) (dnp no) (fields_autoplaced)
     (property "Reference" "L1" (at 94.615 55.88 90)
       (effects (font (size 1.27 1.27)))
@@
   )
   (symbol (lib_id "Device:C") (at 52.705 80.645 0) (unit 1)
-    (in_bom yes) (on_board yes) (dnp no) (fields_autoplaced)
+    (in_bom no) (on_board yes) (dnp no) (fields_autoplaced)
     (property "Reference" "C60" (at 55.88 78.4859 0)
       (effects (font (size 1.27 1.27)) (justify left))
@@
   )
   (symbol (lib_id "Connector:Conn_01x06_Male") (at 28.194 145.796 0) (unit 1)
-    (in_bom yes) (on_board yes) (dnp no) (fields_autoplaced)
+    (in_bom no) (on_board yes) (dnp no) (fields_autoplaced)
     (property "Reference" "J201" (at 28.829 135.89 0)
       (effects (font (size 1.27 1.27)))
@@
   )
   (symbol (lib_id "Device:C") (at 147.32 80.645 0) (unit 1)
-    (in_bom yes) (on_board yes) (dnp no)
+    (in_bom no) (on_board yes) (dnp no)
     (property "Reference" "C55" (at 150.495 78.74 0)
       (effects (font (size 1.27 1.27)) (justify left))
@@
   )
   (symbol (lib_id "Device:C_Small") (at 67.945 104.775 0) (unit 1)
-    (in_bom yes) (on_board yes) (dnp no) (fields_autoplaced)
+    (in_bom no) (on_board yes) (dnp no) (fields_autoplaced)
     (property "Reference" "C57" (at 70.485 103.5112 0)
       (effects (font (size 1.27 1.27)) (justify left))
@@
   )
   (symbol (lib_id "Device:R_Small") (at 130.81 81.915 0) (unit 1)
-    (in_bom yes) (on_board yes) (dnp no)
+    (in_bom no) (on_board yes) (dnp no)
     (property "Reference" "R94" (at 132.08 80.645 0)
       (effects (font (size 1.27 1.27)) (justify left))
@@
   )
   (symbol (lib_id "Device:C") (at 120.65 80.645 0) (unit 1)
-    (in_bom yes) (on_board yes) (dnp no)
+    (in_bom no) (on_board yes) (dnp no)
     (property "Reference" "C56" (at 123.825 78.4859 0)
       (effects (font (size 1.27 1.27)) (justify left))
@@
   )
   (symbol (lib_id "Device:R_Small") (at 139.065 88.9 0) (unit 1)
-    (in_bom yes) (on_board yes) (dnp no)
+    (in_bom no) (on_board yes) (dnp no)
     (property "Reference" "R96" (at 140.335 87.63 0)
       (effects (font (size 1.27 1.27)) (justify left))
@@
   )
   (symbol (lib_id "Device:R_Small") (at 130.81 94.615 0) (unit 1)
-    (in_bom yes) (on_board yes) (dnp no)
+    (in_bom no) (on_board yes) (dnp no)
     (property "Reference" "R95" (at 132.08 93.345 0)
       (effects (font (size 1.27 1.27)) (justify left))
